Commit message: Make the final rig the rig, and teach every gate the steel it stands in
FLEET is now the drawing's three arms — 13 upright on the table, 31 hanging
at h=0.922, 2 on the wall plate with J1 horizontal (a mount this stack never
had; its ready pose is derived and validator-clean).  The six-arm layout
survives verbatim as FLEET_SIXARM, and every module that used to reach for
the module-level registry takes a fleet argument instead, so the legacy
tests run the legacy rig explicitly and bit-identically.

The frame is no longer a proxy: 35 verified boxes from rig_final gate the
lattice, the validator, the atlas and the veto — planner-side by an exact
convex ternary search per capsule, scene_check-side by its own sampling +
Lipschitz derivation, and the two are held together by tests.  The pen
capsule grows to the holder CAD's union envelope (r 0.05), the URDFs carry
the extracted holder mesh on every hand, and the fingers close to the
CAD's 28.5 mm.

The gate caught its first regression before the rig exists: the legacy
inverted ready pose at this rig's height puts the pen 6.6 mm THROUGH the
paper and the elbow 18 mm from the boom.  Both arms that needed one got a
new hover pose, and the refusal of the old one is now a pinned test.

90 tests green, pydrake load + FK checks green.

Co-Authored-By: Claude Fable 5 <noreply@anthropic.com>
Claude-Session: https://claude.ai/code/session_01TYL3Cueh7sskNU8Uz21h7x

File: assets/final_rig/environment.urdf (robot description, URDF)
Before this commit: robot aris_final_rig_env, 36 links, 35 joints
Links:
- added link frame_paper_curl; collision box size=0.125 1.701 0.03; visual box size=0.125 1.701 0.03
- link frame_device_B1: geometry collision box size=0.242 0.1478 0.0978; visual box size=0.242 0.1478 0.0978
- link frame_device_B2: geometry collision box size=0.242 0.1478 0.0978; visual box size=0.242 0.1478 0.0978
- link frame_device_F1: geometry collision box size=0.242 0.147 0.0978; visual box size=0.242 0.147 0.0978
- link frame_device_F2: geometry collision box size=0.242 0.147 0.0978; visual box size=0.242 0.147 0.0978
- link frame_device_L1: geometry collision box size=0.147 0.242 0.0978; visual box size=0.147 0.242 0.0978
- link frame_device_L2: geometry collision box size=0.147 0.242 0.0978; visual box size=0.147 0.242 0.0978
- link frame_device_R1: geometry collision box size=0.148 0.242 0.0978; visual box size=0.148 0.242 0.0978
- link frame_device_R2: geometry collision box size=0.148 0.242 0.0978; visual box size=0.148 0.242 0.0978
- link frame_down_boom_E: geometry collision box size=0.077 0.1524 0.7369; visual box size=0.077 0.1524 0.7369
- link frame_down_boom_W: geometry collision box size=0.0772 0.1524 0.7369; visual box size=0.0772 0.1524 0.7369
- link frame_down_gusset_E: geometry collision box size=0.2044 0.1524 0.2035; visual box size=0.2044 0.1524 0.2035
- link frame_down_gusset_W: geometry collision box size=0.204 0.1524 0.2035; visual box size=0.204 0.1524 0.2035
- link frame_feed_roll: geometry collision box size=0.215 1.765 0.206; visual box size=0.215 1.765 0.206
- link frame_guide_rods: geometry collision box size=0.053 1.739 0.0395; visual box size=0.053 1.739 0.0395
- link frame_side_boom: geometry collision box size=0.0767 0.1524 0.737; visual box size=0.0767 0.1524 0.737
- link frame_side_gusset: geometry collision box size=0.204 0.1524 0.2035; visual box size=0.204 0.1524 0.2035
- link frame_table_block: geometry collision box size=2.1924 2.0908 0.63468; visual box size=2.1924 2.0908 0.63468
- link frame_top_slab: geometry collision box size=2.185 2.0828 0.0762; visual box size=2.185 2.0828 0.0762
Joints:
- added joint frame_paper_curl_weld: type fixed, parent world, child frame_paper_curl

File: assets/final_rig/installation.urdf (robot description, URDF)
Before this commit: robot aris_final_rig, 72 links, 71 joints
Links:
- added link arm13_pen_holder; collision cylinder length=0.243 radius=0.05; visual mesh filename=meshes/penholder_rig10_panda_hand_frame.stl
- added link arm2_pen_holder; collision cylinder length=0.243 radius=0.05; visual mesh filename=meshes/penholder_rig10_panda_hand_frame.stl
- added link arm31_pen_holder; collision cylinder length=0.243 radius=0.05; visual mesh filename=meshes/penholder_rig10_panda_hand_frame.stl
- added link frame_paper_curl; collision box size=0.125 1.701 0.03; visual box size=0.125 1.701 0.03
- link frame_device_B1: geometry collision box size=0.242 0.1478 0.0978; visual box size=0.242 0.1478 0.0978
- link frame_device_B2: geometry collision box size=0.242 0.1478 0.0978; visual box size=0.242 0.1478 0.0978
- link frame_device_F1: geometry collision box size=0.242 0.147 0.0978; visual box size=0.242 0.147 0.0978
- link frame_device_F2: geometry collision box size=0.242 0.147 0.0978; visual box size=0.242 0.147 0.0978
- link frame_device_L1: geometry collision box size=0.147 0.242 0.0978; visual box size=0.147 0.242 0.0978
- link frame_device_L2: geometry collision box size=0.147 0.242 0.0978; visual box size=0.147 0.242 0.0978
- link frame_device_R1: geometry collision box size=0.148 0.242 0.0978; visual box size=0.148 0.242 0.0978
- link frame_device_R2: geometry collision box size=0.148 0.242 0.0978; visual box size=0.148 0.242 0.0978
- link frame_down_boom_E: geometry collision box size=0.077 0.1524 0.7369; visual box size=0.077 0.1524 0.7369
- link frame_down_boom_W: geometry collision box size=0.0772 0.1524 0.7369; visual box size=0.0772 0.1524 0.7369
- link frame_down_gusset_E: geometry collision box size=0.2044 0.1524 0.2035; visual box size=0.2044 0.1524 0.2035
- link frame_down_gusset_W: geometry collision box size=0.204 0.1524 0.2035; visual box size=0.204 0.1524 0.2035
- link frame_feed_roll: geometry collision box size=0.215 1.765 0.206; visual box size=0.215 1.765 0.206
- link frame_guide_rods: geometry collision box size=0.053 1.739 0.0395; visual box size=0.053 1.739 0.0395
- link frame_side_boom: geometry collision box size=0.0767 0.1524 0.737; visual box size=0.0767 0.1524 0.737
- link frame_side_gusset: geometry collision box size=0.204 0.1524 0.2035; visual box size=0.204 0.1524 0.2035
- link frame_table_block: geometry collision box size=2.1924 2.0908 0.63468; visual box size=2.1924 2.0908 0.63468
- link frame_top_slab: geometry collision box size=2.185 2.0828 0.0762; visual box size=2.185 2.0828 0.0762
Joints:
- added joint arm13_pen_holder_weld: type fixed, parent arm13_panda_hand, child arm13_pen_holder
- added joint arm2_pen_holder_weld: type fixed, parent arm2_panda_hand, child arm2_pen_holder
- added joint arm31_pen_holder_weld: type fixed, parent arm31_panda_hand, child arm31_pen_holder
- added joint frame_paper_curl_weld: type fixed, parent world, child frame_paper_curl
- joint arm13_panda_finger_joint1: origin xyz=0 0.008 0.0584 rpy=0 0 0 -> xyz=0 0.0285 0.0584 rpy=0 0 0
- joint arm13_panda_finger_joint2: origin xyz=0 -0.008 0.0584 rpy=0 0 0 -> xyz=0 -0.0285 0.0584 rpy=0 0 0
- joint arm2_panda_finger_joint1: origin xyz=0 0.008 0.0584 rpy=0 0 0 -> xyz=0 0.0285 0.0584 rpy=0 0 0
- joint arm2_panda_finger_joint2: origin xyz=0 -0.008 0.0584 rpy=0 0 0 -> xyz=0 -0.0285 0.0584 rpy=0 0 0
- joint arm31_panda_finger_joint1: origin xyz=0 0.008 0.0584 rpy=0 0 0 -> xyz=0 0.0285 0.0584 rpy=0 0 0
- joint arm31_panda_finger_joint2: origin xyz=0 -0.008 0.0584 rpy=0 0 0 -> xyz=0 -0.0285 0.0584 rpy=0 0 0
