Commit message: Hang it 9 cm higher: it buys back the canvas, not the fleet
Re-certifies the all-ceiling rig at h = 0.925 and 0.940 against the adopted
0.850, end to end under the corrected capsules -- parks re-derived, atlas
re-swept, URDF regenerated, placement re-searched, the CSAIL logo re-allocated
and re-conducted in every mode the conductor has -- and ships 0.940.

                    0.850      0.925      0.940     0.940 @ pitch 0.65
  union strict-GO   87.00 %    91.10 %    90.70 %   91.95 %
  >=2 arms          37.14 %    34.43 %    33.85 %   34.61 %
  sigma p1          0.1513     0.1516     0.1468    --
  pair clearance    80.3 %     82.8 %     83.6 %    --   (worst of 15)
  best park-vs-ink  10 mm      61 mm      72 mm     68 mm
  6-mover           refused    refused    refused   refused
  partner-disjoint  refused    refused    refused   refused
  solo              refused    refused    22.6 %    26.1 %

HEIGHT HELPS AND DOES NOT SOLVE IT.  Union coverage gains 4 pp, the dead area
falls by a third, every pair's clearance improves -- and the number that
decides whether anything runs at all climbs monotonically: how far the best
park set can get from every other arm's certified ink goes 10 -> 61 -> 72 mm
against the 80 mm the conductor asks.  At 0.850 and 0.925 the shortfall is
total and the rig draws NOTHING; at 0.940 one solo phase clears.  0.940 is not
the coverage optimum (0.925 beats it by 0.4 pp) and it is shipped anyway,
because it is the only height of the three that produces a certified programme.

IT IS NOT THE MARGIN.  Re-conducting with calib cut to zero -- margin 0.08 ->
0.05, which is what a base survey buys -- returns the same phase and the same
22.6 %.  IT IS THE MIDDLE ROW: a park's radius saturates (the hover point is
clipped into the sheet, so past ~0.55 m every candidate lands on the same xy)
and its hover saturates (arms 31 and 71 certify nothing above 0.40-0.50 m).
Two arms over the middle of a 1.80 m canvas have nowhere to stand that is not
inside somebody's drawing, and the conductor names it: "the impossible indices
are INK: arm 13 segment(s) [11] -- no order fixes that, only a different
allocation".

PARK_GRID_PROPOSED is re-searched, on the criterion that turned out to matter:
7 radii x 10 hovers per arm, ranked on clearance to every OTHER arm's
certified drawing poses rather than on its own arm's flyability.  The winners
park 0.30-0.50 m over the paper where the 0.850 rig parked at 0.10-0.20.

PROFILES_LAT gains an ("inv", 0.940) row measured off the real six-arm atlas
rather than off the box-free probe the other rows come from, and PAIR_WINDOW
follows it from (0.40, 0.64) to (0.26, 0.73) -- which is how pitch 0.65 and
0.70 became admissible, and why the 0.65 column above is in the table.  Pitch
is a build-sheet number and is NOT changed here.

Also: a re-sequencing refusal is a phase verdict now.  `resequence` prices
segment orders against the transit router and can come back with no finite
tour at all; that used to propagate out of `build` as an unhandled RuntimeError
and take the whole programme with it, where the identical statement from the
conductor one stage later is caught and skipped.  Same dial, same place.

Shipped programme: one phase (arm 31, 10 segments, 2.388 m), makespan 37.6 s,
zero conducted pause, scene_check PASS, min inter-arm 146.2 mm, column
144.1 mm, frame 51.2 mm, paper chain 108.4 mm.  out/csail_proposed_h094.{html,
zip} (33.0 / 16.7 MB).  264 passed, 7 skipped.

docs/BUILD_SHEET.md is deliberately untouched: its 1 is a number the rig
owner revises, and this commit is the evidence for revising it, not the
revision.

Co-Authored-By: Claude Opus 5 <noreply@anthropic.com>
Claude-Session: https://claude.ai/code/session_01TYL3Cueh7sskNU8Uz21h7x

File: assets/proposed_rig/environment.urdf (robot description, URDF)
Before this commit: robot aris_proposed_rig_env, 15 links, 14 joints
Links:
- link mount13_boom: geometry collision box size=0.2 0.2 1.35; visual cylinder length=1.35 radius=0.1
- link mount17_boom: geometry collision box size=0.2 0.2 1.35; visual cylinder length=1.35 radius=0.1
- link mount2_boom: geometry collision box size=0.2 0.2 1.35; visual cylinder length=1.35 radius=0.1
- link mount31_boom: geometry collision box size=0.2 0.2 1.35; visual cylinder length=1.35 radius=0.1
- link mount71_boom: geometry collision box size=0.2 0.2 1.35; visual cylinder length=1.35 radius=0.1
- link mount97_boom: geometry collision box size=0.2 0.2 1.35; visual cylinder length=1.35 radius=0.1

File: assets/proposed_rig/installation.urdf (robot description, URDF)
Before this commit: robot aris_proposed_rig, 123 links, 122 joints
Links:
- link mount13_boom: geometry collision box size=0.2 0.2 1.35; visual cylinder length=1.35 radius=0.1
- link mount17_boom: geometry collision box size=0.2 0.2 1.35; visual cylinder length=1.35 radius=0.1
- link mount2_boom: geometry collision box size=0.2 0.2 1.35; visual cylinder length=1.35 radius=0.1
- link mount31_boom: geometry collision box size=0.2 0.2 1.35; visual cylinder length=1.35 radius=0.1
- link mount71_boom: geometry collision box size=0.2 0.2 1.35; visual cylinder length=1.35 radius=0.1
- link mount97_boom: geometry collision box size=0.2 0.2 1.35; visual cylinder length=1.35 radius=0.1
Joints:
- joint arm13_mount_weld: origin xyz=0.5967 0.605106667 0.85 rpy=3.141592654 0 3.141592654 -> xyz=0.5967 0.605106667 0.94 rpy=3.141592654 0 3.141592654
- joint arm17_mount_weld: origin xyz=1.2067 0.605106667 0.85 rpy=3.141592654 0 3.141592654 -> xyz=1.2067 0.605106667 0.94 rpy=3.141592654 0 3.141592654
- joint arm2_mount_weld: origin xyz=0.5967 3.025533333 0.85 rpy=3.141592654 0 3.141592654 -> xyz=0.5967 3.025533333 0.94 rpy=3.141592654 0 3.141592654
- joint arm31_mount_weld: origin xyz=0.5967 1.81532 0.85 rpy=3.141592654 0 3.141592654 -> xyz=0.5967 1.81532 0.94 rpy=3.141592654 0 3.141592654
- joint arm71_mount_weld: origin xyz=1.2067 1.81532 0.85 rpy=3.141592654 0 3.141592654 -> xyz=1.2067 1.81532 0.94 rpy=3.141592654 0 3.141592654
- joint arm97_mount_weld: origin xyz=1.2067 3.025533333 0.85 rpy=3.141592654 0 3.141592654 -> xyz=1.2067 3.025533333 0.94 rpy=3.141592654 0 3.141592654
