Commit message: The pen leaves through the cap, and now the model does too
`penholder22_T_hand` set `Xh = -u`: the housing's +X pointed away from the
tip, so the 17.00 mm tail land sat 55.099 mm toward the paper and the cap
30.001 mm back toward the wrist.  §7c has said the pen leaves through the CAP
since 2026-09-02 and deferred the fix as a re-certification.  This is the
re-certification.

Re-derived from `Natural hold assembly - closed.SLDASM` itself, not from the
prose: along that assembly's bore the parts run cap 1017.121..1028.558,
sleeve 1020.121..1060.221, SPRING 1060.121..1098.919, housing tail face
1102.221 — the spring is at the end away from the cap and pushes the pen
toward it, which is the tool's whole compliance.  Its pencil spans
1000.121..1174.735: 17.000 mm of sharpened point past the cap's outer face and
72.514 mm of blunt tail past the tail face, which is what its own preview
draws.  17.00 will not pass a 19.05 spring and does not touch a 7 mm stick.
And the grip is 25.001 mm from the housing's cap end against 55.099 from its
tail, the same 25 mm docs/FINAL_RIG.md read independently.

`Xh = u` — a 180 deg rotation about the post axis and nothing else.  The post
axis is still y_hand, the grip centre is still the TCP, the bore is still the
planner's 45 deg ray, and THE PEN TIP DOES NOT MOVE: check_system_model still
reports the same worst 5.259e-12 m over 25 configs x 6 arms, digit for digit,
and a new test pins it.  Grip-to-exit becomes +30.001 mm (the cap's outer
face; 25.001 to the housing's end face plus the 5.000 the cap stands proud),
so the planner's 155.563 mm tip now needs 125.562 mm of graphite past the cap
and the 23 deg CAD lean needs 89.499.  §7c's 130.5 / 94.5 were measured to the
housing's end face; both faces are now named wherever the number appears.

THE PENCIL TAIL IS A BODY NOW.  It was in the assembly, in the preview, and
nowhere in this model: 72.514 mm of stick out the tail face, pointing at the
wrist.  `penholder22_tail` places it with its own envelope cylinder fitted the
way `env_cylinders` are, escape proved at 0.0 m on every generator run, so the
tool's collision model is four cylinders rather than three.  Measured 72.514
is the assembly's; ASSUMED is that this build shows the same overhang, and the
price is written down — a stick that still shows it is 283.176 mm long, and
the assembly's own 174.614 mm pencil pushed to this tip ends 36.049 mm inside
the barrel with no tail at all.

WHAT THE RE-CERTIFICATION COST, measured, absorbed nowhere.  scene_check on
out/csail_schedule_h094_v14.* is BIT-IDENTICAL before and after and still
PASSes (80.73 mm inter-arm against an 80 mm margin, arms 13-17), because the
planner's tool is the two-capsule L and that did not move.  But the L no
longer CONTAINS the holder: housing+cap escape its r = 0.050 by 6.546 mm
(bracket r 0.0565 needed) where the end-for-end placement was contained by
1.720 mm, and the tail escapes by 77.661 mm (r 0.1277).  Re-run at those radii
the same programme fails the 80 mm gate — 79.12 mm, then -18.21 mm, and the
50 mm frame gate too.  No capsule radius, gate constant, layout number or
planner semantic was touched; the escape is reported in 7c, in the manifest
and by `collision_audit --part tool` on every run.  Self-collision at the six
parks: the tail clears the hand shell by 43.02 mm, link7's by 45.88 and the
fingers by 32.56, and sits +3.36 mm off the hand.0 capsule and +12.83 mm off
link7.1 — under SELF_PLAN_MARGIN, in pairs selfcoll deliberately does not
watch (chain distance 0 and 1, against WATCH_CHAIN_D = 4), so no gate flips.

assets/proposed_rig/ is no longer untouched, and its README says so: leaving a
body known to be on backwards in the tree every certified number was checked
against is worse than the churn.  Everything else there is unmoved.

test_regeneration_is_byte_stable is green again as a side effect: the 48 and
150 ULP lines of §10 were re-measured against the old code in this environment
first (they reproduce exactly) so nothing hid inside the larger diff.

New: a `holder_side` render, straight down the hand's x axis with up = -z_hand
— fingers across the frame, barrel and tail above the grip, cap and graphite
below it.  The shot that would have caught this a day earlier.

Co-Authored-By: Claude Opus 5 <noreply@anthropic.com>
Claude-Session: https://claude.ai/code/session_01TYL3Cueh7sskNU8Uz21h7x

File: assets/proposed_rig/installation.urdf (robot description, URDF)
Before this commit: robot aris_proposed_rig, 123 links, 122 joints
Links:
- link arm13_pen_holder: geometry collision cylinder length=0.0115 radius=0.0181; collision cylinder length=0.035 radius=0.0136
- link arm13_pen_lead: geometry collision cylinder length=0.125562492 radius=0.005; visual cylinder length=0.125562492 radius=0.0035
- link arm17_pen_holder: geometry collision cylinder length=0.0115 radius=0.0181; collision cylinder length=0.035 radius=0.0136
- link arm17_pen_lead: geometry collision cylinder length=0.125562492 radius=0.005; visual cylinder length=0.125562492 radius=0.0035
- link arm2_pen_holder: geometry collision cylinder length=0.0115 radius=0.0181; collision cylinder length=0.035 radius=0.0136
- link arm2_pen_lead: geometry collision cylinder length=0.125562492 radius=0.005; visual cylinder length=0.125562492 radius=0.0035
- link arm31_pen_holder: geometry collision cylinder length=0.0115 radius=0.0181; collision cylinder length=0.035 radius=0.0136
- link arm31_pen_lead: geometry collision cylinder length=0.125562492 radius=0.005; visual cylinder length=0.125562492 radius=0.0035
- link arm71_pen_holder: geometry collision cylinder length=0.0115 radius=0.0181; collision cylinder length=0.035 radius=0.0136
- link arm71_pen_lead: geometry collision cylinder length=0.125562492 radius=0.005; visual cylinder length=0.125562492 radius=0.0035
- link arm97_pen_holder: geometry collision cylinder length=0.0115 radius=0.0181; collision cylinder length=0.035 radius=0.0136
- link arm97_pen_lead: geometry collision cylinder length=0.125562492 radius=0.005; visual cylinder length=0.125562492 radius=0.0035

File: assets/system_model/installation.urdf (robot description, URDF)
Before this commit: robot aris_system_model, 186 links, 185 joints
Links:
- link arm13_pen_holder: geometry collision cylinder length=0.01150000000000001 radius=0.0181; collision cylinder length=0.035 radius=0.0136
- link arm13_pen_lead: geometry collision cylinder length=0.12556249186104046 radius=0.005; visual cylinder length=0.12556249186104046 radius=0.0035
- link arm17_pen_holder: geometry collision cylinder length=0.01150000000000001 radius=0.0181; collision cylinder length=0.035 radius=0.0136
- link arm17_pen_lead: geometry collision cylinder length=0.12556249186104046 radius=0.005; visual cylinder length=0.12556249186104046 radius=0.0035
- link arm2_pen_holder: geometry collision cylinder length=0.01150000000000001 radius=0.0181; collision cylinder length=0.035 radius=0.0136
- link arm2_pen_lead: geometry collision cylinder length=0.12556249186104046 radius=0.005; visual cylinder length=0.12556249186104046 radius=0.0035
- link arm31_pen_holder: geometry collision cylinder length=0.01150000000000001 radius=0.0181; collision cylinder length=0.035 radius=0.0136
- link arm31_pen_lead: geometry collision cylinder length=0.12556249186104046 radius=0.005; visual cylinder length=0.12556249186104046 radius=0.0035
- link arm71_pen_holder: geometry collision cylinder length=0.01150000000000001 radius=0.0181; collision cylinder length=0.035 radius=0.0136
- link arm71_pen_lead: geometry collision cylinder length=0.12556249186104046 radius=0.005; visual cylinder length=0.12556249186104046 radius=0.0035
- link arm97_pen_holder: geometry collision cylinder length=0.01150000000000001 radius=0.0181; collision cylinder length=0.035 radius=0.0136
- link arm97_pen_lead: geometry collision cylinder length=0.12556249186104046 radius=0.005; visual cylinder length=0.12556249186104046 radius=0.0035

File: assets/system_model/installation_capsules.urdf (robot description, URDF)
Before this commit: robot aris_system_model_capsule, 186 links, 185 joints
Links:
- link arm13_panda_link3: geometry collision {http://drake.mit.edu}capsule length=0.11621243479077442 radius=0.062; collision {http://drake.mit.edu}capsule length=0.1294729315339697 radius=0.059
- link arm13_panda_link4: geometry collision {http://drake.mit.edu}capsule length=0.11444203773089677 radius=0.062; collision {http://drake.mit.edu}capsule length=0.128346756873713 radius=0.077
- link arm13_pen_holder: geometry collision cylinder length=0.01150000000000001 radius=0.0181; collision cylinder length=0.035 radius=0.0136
- link arm13_pen_lead: geometry collision cylinder length=0.12556249186104046 radius=0.005; visual cylinder length=0.12556249186104046 radius=0.0035
- link arm17_panda_link3: geometry collision {http://drake.mit.edu}capsule length=0.11621243479077442 radius=0.062; collision {http://drake.mit.edu}capsule length=0.1294729315339697 radius=0.059
- link arm17_panda_link4: geometry collision {http://drake.mit.edu}capsule length=0.11444203773089677 radius=0.062; collision {http://drake.mit.edu}capsule length=0.128346756873713 radius=0.077
- link arm17_pen_holder: geometry collision cylinder length=0.01150000000000001 radius=0.0181; collision cylinder length=0.035 radius=0.0136
- link arm17_pen_lead: geometry collision cylinder length=0.12556249186104046 radius=0.005; visual cylinder length=0.12556249186104046 radius=0.0035
- link arm2_panda_link3: geometry collision {http://drake.mit.edu}capsule length=0.11621243479077442 radius=0.062; collision {http://drake.mit.edu}capsule length=0.1294729315339697 radius=0.059
- link arm2_panda_link4: geometry collision {http://drake.mit.edu}capsule length=0.11444203773089677 radius=0.062; collision {http://drake.mit.edu}capsule length=0.128346756873713 radius=0.077
- link arm2_pen_holder: geometry collision cylinder length=0.01150000000000001 radius=0.0181; collision cylinder length=0.035 radius=0.0136
- link arm2_pen_lead: geometry collision cylinder length=0.12556249186104046 radius=0.005; visual cylinder length=0.12556249186104046 radius=0.0035
- link arm31_panda_link3: geometry collision {http://drake.mit.edu}capsule length=0.11621243479077442 radius=0.062; collision {http://drake.mit.edu}capsule length=0.1294729315339697 radius=0.059
- link arm31_panda_link4: geometry collision {http://drake.mit.edu}capsule length=0.11444203773089677 radius=0.062; collision {http://drake.mit.edu}capsule length=0.128346756873713 radius=0.077
- link arm31_pen_holder: geometry collision cylinder length=0.01150000000000001 radius=0.0181; collision cylinder length=0.035 radius=0.0136
- link arm31_pen_lead: geometry collision cylinder length=0.12556249186104046 radius=0.005; visual cylinder length=0.12556249186104046 radius=0.0035
- link arm71_panda_link3: geometry collision {http://drake.mit.edu}capsule length=0.11621243479077442 radius=0.062; collision {http://drake.mit.edu}capsule length=0.1294729315339697 radius=0.059
- link arm71_panda_link4: geometry collision {http://drake.mit.edu}capsule length=0.11444203773089677 radius=0.062; collision {http://drake.mit.edu}capsule length=0.128346756873713 radius=0.077
- link arm71_pen_holder: geometry collision cylinder length=0.01150000000000001 radius=0.0181; collision cylinder length=0.035 radius=0.0136
- link arm71_pen_lead: geometry collision cylinder length=0.12556249186104046 radius=0.005; visual cylinder length=0.12556249186104046 radius=0.0035
- link arm97_panda_link3: geometry collision {http://drake.mit.edu}capsule length=0.11621243479077442 radius=0.062; collision {http://drake.mit.edu}capsule length=0.1294729315339697 radius=0.059
- link arm97_panda_link4: geometry collision {http://drake.mit.edu}capsule length=0.11444203773089677 radius=0.062; collision {http://drake.mit.edu}capsule length=0.128346756873713 radius=0.077
- link arm97_pen_holder: geometry collision cylinder length=0.01150000000000001 radius=0.0181; collision cylinder length=0.035 radius=0.0136
- link arm97_pen_lead: geometry collision cylinder length=0.12556249186104046 radius=0.005; visual cylinder length=0.12556249186104046 radius=0.0035

File: assets/system_model/installation_fatfingers.urdf (robot description, URDF)
Before this commit: robot aris_system_model_fatfingers, 186 links, 185 joints
Links:
- link arm13_pen_holder: geometry collision cylinder length=0.01150000000000001 radius=0.0181; collision cylinder length=0.035 radius=0.0136
- link arm13_pen_lead: geometry collision cylinder length=0.12556249186104046 radius=0.005; visual cylinder length=0.12556249186104046 radius=0.0035
- link arm17_pen_holder: geometry collision cylinder length=0.01150000000000001 radius=0.0181; collision cylinder length=0.035 radius=0.0136
- link arm17_pen_lead: geometry collision cylinder length=0.12556249186104046 radius=0.005; visual cylinder length=0.12556249186104046 radius=0.0035
- link arm2_pen_holder: geometry collision cylinder length=0.01150000000000001 radius=0.0181; collision cylinder length=0.035 radius=0.0136
- link arm2_pen_lead: geometry collision cylinder length=0.12556249186104046 radius=0.005; visual cylinder length=0.12556249186104046 radius=0.0035
- link arm31_pen_holder: geometry collision cylinder length=0.01150000000000001 radius=0.0181; collision cylinder length=0.035 radius=0.0136
- link arm31_pen_lead: geometry collision cylinder length=0.12556249186104046 radius=0.005; visual cylinder length=0.12556249186104046 radius=0.0035
- link arm71_pen_holder: geometry collision cylinder length=0.01150000000000001 radius=0.0181; collision cylinder length=0.035 radius=0.0136
- link arm71_pen_lead: geometry collision cylinder length=0.12556249186104046 radius=0.005; visual cylinder length=0.12556249186104046 radius=0.0035
- link arm97_pen_holder: geometry collision cylinder length=0.01150000000000001 radius=0.0181; collision cylinder length=0.035 radius=0.0136
- link arm97_pen_lead: geometry collision cylinder length=0.12556249186104046 radius=0.005; visual cylinder length=0.12556249186104046 radius=0.0035
