Commit message: The pen was seven centimetres too long, and the barrel behind the grip is what says the lean cannot be 23 degrees
Pete photographed the real gripper.  Three things in this model were checked
against it; one was already right, one was wrong by 72 mm, and one that had
been called an open question for two days turned out to be closed by geometry
nobody had looked at.

THE BLADES ARE MOUNTED THE WAY THIS MODEL HAS THEM, and there was never
another option.  The photo shows each Fat Franka Finger's foot outboard at the
carriage, the web slanting down and inward, the plate inboard of the foot, and
the two blades converging toward the paper.  That is `rig_final.FATFINGER`
exactly: in `panda_hand` at `FAT_FINGER_FIX` the feet stand 70.867 mm apart
over z 62.24..76.24 and the plates 55.168 mm apart over z 94.24..112.24, a V
closing 15.7 mm over 50 mm of finger.  The "10.65 mm OUTBOARD" that reads like
the opposite is measured from the STOCK GRIP PLANE, a different datum from the
foot: the blade is 15.85 mm thick from carriage face to contact face where the
stock finger is 26.4 mm from carriage face to grip plane, and that difference
IS the 10.65.  The mirror — the foot's inner face on the carriage, web
outward — puts the contact plate at link y 34.350 instead of 10.650, so two
plates sit 68.700 mm apart at q = 0 and closing them on a 50 mm post needs
q = -9.350 mm.  It cannot grip this holder at any joint value.  NOTHING MOVED
IN THE BLADE MODEL, and a new test pins both halves of that with the photo's
own description in its docstring.

So the width table is the same six it was, and the photo cuts it to two: no
fingertip is fitted, so every row that seats one is out.  EXPECT 0.0339 off
the robot (the rib lands first, which is what the URDF draws) or 0.0287 (the
plates flat, if the post is seated distal of the rib).  Both FAIL the GUI's
`grasp(0.0432, epsilon_inner=0.0)` — not a contradiction, because that menu
path falls back to a move-close, but it is the open item.  Read the other way,
`width` is a ruler: a reading of w puts the contact face (50 - 1000 w)/2 mm
outboard of the stock grip plane, so 0.0432 would mean the foot is bolted
7.2 mm further inboard than modelled.  That is the one thing about the blade
the photo could not settle, and it is worth 16 mm of `width`.

23 DEGREES IS RULED OUT, BY THE HAND.  The mount post sits 55.099 mm from the
housing's tail face, so 55.1 mm of barrel stands BEHIND the grip pointing at
the wrist — a body this model did not have until the 7c flip gave it one — and
there are 37.4 mm between the grip and the hand's underside.  Swept against
the convex hull of the manufacturer's own `hand.obj` collision shell, the raw
housing STL is INSIDE the hand at every lean below 35.17 deg: -18.79 mm at 10,
-11.90 at 23, -0.16 at 35, +6.16 at 45.  A 23 deg build would pass twelve
millimetres of printed barrel through the gripper's casting.  The photo is
what makes the argument bite: with no fingertip seated in the post's socket
nothing transmits the housing's 23 deg clocking, so the lean is set by hand at
grasp time — and the hand only admits 45.  This is the first argument for the
planner's ray that is about the hardware rather than about the planner, and it
overturns 7a's "verdict: the pen leans 23 deg".

AND THE TIP MOVED, 72.348 mm.  "Just have the pen protruding out the bottom of
those finger extensions by ca 5 cm."  The blades' contact plates end at
`panda_hand` z = 0.1122421, so the tip is at 0.1622421 and, from the hand TCP:

    PEN_LEAN_HOLDER = 45 deg            forced by the hand, above
    PEN_EXT_HOLDER  = 0.1622421 - 0.1034 = 0.0588421 m      (NEW CONSTANT)
    PEN_LAT_HOLDER  = PEN_EXT_HOLDER * tan 45 deg = 0.0588421 m   (was 0.110)

Reach from the grip 155.563 -> 83.215 mm; graphite past the cap's outer face
125.562 -> 53.214 mm, which reads 37.6 mm in the photo's own foreshortened
view against the 20-40 mm it shows.  The 72.514 mm pencil tail stops being an
embarrassment: 72.514 + 85.100 + 53.214 = 210.8 mm of stick, where the old tip
asked for 283.2 mm and no 7 mm graphite is that long.  THE HOLDER BODY DOES
NOT MOVE BY A PICOMETRE — its placement is fixed by the ray's DIRECTION and by
the grip centre, both unchanged — so both hand-frame housing meshes are
byte-identical across this commit and every escape 7c measured still stands.

BOTH HALVES OF THE TOOL SWITCH NOW.  `activate_tool` set only `PEN_LAT`, so a
lateral run drew the holder's 45 deg ray out to the INLINE pen's axial 0.110 —
a tool that exists nowhere.  It did not matter while the two numbers were both
0.110.  `PEN_EXT_ACTIVE` and `ext_of` are the twins of `PEN_LAT` and `lat_of`,
`activate_tool` sets both, and every `pen_ext=PEN_EXT` default in the package
(81 of them, in 17 modules) is `pen_ext=None` instead — because a default
written as a module constant binds the inline pen AT IMPORT and no later
`activate_tool` can reach it.  Sixteen sites that did arithmetic on `pen_ext`
resolve through `ext_of` now; `ArmSpec.pen`, `stroke_api.DEFAULTS` and
`certified_ready_pose` follow the active tool rather than a literal.  With the
inline tool active — the repo default — `ext_of(None)` is 0.110 and every
inline number is unchanged.  A plan result records `pen_ext` alongside
`pen_lat`, because a plan that names one half of its tool does not name its
tool.

`certified_ready_pose` was one of the mixed-tool sites and it is the one that
bit: it took `pen_lat` explicitly and let the axial half fall through, and at
the new pair that mixture certifies no pose at all for arm 71.

THE INLINE PEN IS UNTOUCHED, AND IT IS THE ONLY ONE THAT WAS EVER MEASURED.
`PEN_EXT = 0.110` is a real gate-B touchdown at MZ 0.924 and nothing here
moves it.  The HOLDER's pair never was: `frames.py` has always said
USER-SPECIFIED, and 7a, 7c, 7d, `system_model.OPEN_QUESTIONS`, `rig_final`,
README, DECISIONS, LAYOUT_STUDY, FINAL_RIG and two tests all called it
"gate-validated against a real touchdown".  Every one of them now says what
frames.py says.

WHAT IT COSTS, MEASURED, ABSORBED NOWHERE.  Every certified programme and
atlas in `out/` (CSAIL v14, the feasible-workspace maps, the lateral eval) was
planned at the old tip and is STALE; re-planning them is queued, not done
here.  `Q_PARK_PROPOSED` is stale too and says so at its own definition: run
at the new pair the same grid parks arms 13 and 17 53.7 mm apart, under the
conductor's 80 mm, and the fix is a fresh (radius, hover, bearing) search
against an atlas, not a different assertion.  The six poses as they stand
still pass `check_pose` at the new tool, the fleet holds 250 mm, and the
shorter pen only lifts each tip about 70 mm — safe, but no longer that
function's own output, so `tests/test_layout.py` re-derives them at 0.110 and
says why.  Two numbers in 7c's self-collision table could not be reproduced
and are corrected with the method written down: the corrected housing clears
the manufacturer's hand shell by 6.16 mm (not 49.21) and the pencil tail by
18.36 mm (not 43.02), the tail's closest approach being at its START by the
tail face rather than at its far end, which swings out in hand x and clears by
59.04 mm.  18.4 mm is the model agreeing with the photo's "almost touching",
which the old 43.0 mm did not.

Regenerated: `assets/system_model/` (four URDFs + manifest) and
`assets/proposed_rig/installation.urdf`; the holder meshes in both are
byte-identical.  `check_system_model.py` ALL PASS, worst pen tip 4.779e-12 m
over 25 configs x 6 arms against the NEW tip; `check_proposed_rig_urdf.py` ALL
PASS, worst 9.461e-10 m.  New render `--views photo`: the photograph's own
viewpoint, an oblique from below the hand down its x axis, where the blades
read as a V and the tail is seen standing out at the wrist.

TESTS.  `pytest tests/` less the two files that take 25 minutes each
(`test_balance`, `test_csail`, both of which use the INLINE pen explicitly and
showed no failure before their own timeouts): 346 passed, 24 skipped, 3
failed — and all three of those reproduce at HEAD, unstashed, so this change
adds no failure.  They are `test_draw`'s SVG trace (a numpy cross-product API
change) and `test_planner_robustness`' two FK bit-identity tests (the C++
batch against python at 1e-14 in a rotation).  `test_lateral` is 27 green,
`test_system_model` 55, `test_layout` 26, and `test_merge_spans` caught the
one real miss of the refactor — `paper.py`'s lift memo was still doing
`float(pen_ext)` on a `None`.

docs/SYSTEM_MODEL.md gains 7e, which is the account and two conversion tables:
graphite-past-the-cap -> tip, and measured tip-to-approach-axis -> everything
else, at both leans, with the 23 deg rows marked as arithmetic rather than
candidates.

Co-Authored-By: Claude Opus 5 <noreply@anthropic.com>
Claude-Session: https://claude.ai/code/session_01TYL3Cueh7sskNU8Uz21h7x

File: assets/proposed_rig/installation.urdf (robot description, URDF)
Before this commit: robot aris_proposed_rig, 123 links, 122 joints
Links:
- link arm13_pen_body: geometry collision cylinder length=0.0588421 radius=0.05
- link arm13_pen_bracket: geometry collision cylinder length=0.0588421 radius=0.05
- link arm13_pen_lead: geometry collision cylinder length=0.053214296 radius=0.005; visual cylinder length=0.053214296 radius=0.0035
- link arm17_pen_body: geometry collision cylinder length=0.0588421 radius=0.05
- link arm17_pen_bracket: geometry collision cylinder length=0.0588421 radius=0.05
- link arm17_pen_lead: geometry collision cylinder length=0.053214296 radius=0.005; visual cylinder length=0.053214296 radius=0.0035
- link arm2_pen_body: geometry collision cylinder length=0.0588421 radius=0.05
- link arm2_pen_bracket: geometry collision cylinder length=0.0588421 radius=0.05
- link arm2_pen_lead: geometry collision cylinder length=0.053214296 radius=0.005; visual cylinder length=0.053214296 radius=0.0035
- link arm31_pen_body: geometry collision cylinder length=0.0588421 radius=0.05
- link arm31_pen_bracket: geometry collision cylinder length=0.0588421 radius=0.05
- link arm31_pen_lead: geometry collision cylinder length=0.053214296 radius=0.005; visual cylinder length=0.053214296 radius=0.0035
- link arm71_pen_body: geometry collision cylinder length=0.0588421 radius=0.05
- link arm71_pen_bracket: geometry collision cylinder length=0.0588421 radius=0.05
- link arm71_pen_lead: geometry collision cylinder length=0.053214296 radius=0.005; visual cylinder length=0.053214296 radius=0.0035
- link arm97_pen_body: geometry collision cylinder length=0.0588421 radius=0.05
- link arm97_pen_bracket: geometry collision cylinder length=0.0588421 radius=0.05
- link arm97_pen_lead: geometry collision cylinder length=0.053214296 radius=0.005; visual cylinder length=0.053214296 radius=0.0035
Joints:
- joint arm13_pen_body_weld: origin xyz=0.11 0 0 -> xyz=0.0588421 0 0
- joint arm13_pen_tip_weld: origin xyz=0 0 0.11 -> xyz=0 0 0.0588421
- joint arm17_pen_body_weld: origin xyz=0.11 0 0 -> xyz=0.0588421 0 0
- joint arm17_pen_tip_weld: origin xyz=0 0 0.11 -> xyz=0 0 0.0588421
- joint arm2_pen_body_weld: origin xyz=0.11 0 0 -> xyz=0.0588421 0 0
- joint arm2_pen_tip_weld: origin xyz=0 0 0.11 -> xyz=0 0 0.0588421
- joint arm31_pen_body_weld: origin xyz=0.11 0 0 -> xyz=0.0588421 0 0
- joint arm31_pen_tip_weld: origin xyz=0 0 0.11 -> xyz=0 0 0.0588421
- joint arm71_pen_body_weld: origin xyz=0.11 0 0 -> xyz=0.0588421 0 0
- joint arm71_pen_tip_weld: origin xyz=0 0 0.11 -> xyz=0 0 0.0588421
- joint arm97_pen_body_weld: origin xyz=0.11 0 0 -> xyz=0.0588421 0 0
- joint arm97_pen_tip_weld: origin xyz=0 0 0.11 -> xyz=0 0 0.0588421

File: assets/system_model/installation.urdf (robot description, URDF)
Before this commit: robot aris_system_model, 186 links, 185 joints
Links:
- link arm13_pen_lead: geometry collision cylinder length=0.0532142958585139 radius=0.005; visual cylinder length=0.0532142958585139 radius=0.0035
- link arm17_pen_lead: geometry collision cylinder length=0.0532142958585139 radius=0.005; visual cylinder length=0.0532142958585139 radius=0.0035
- link arm2_pen_lead: geometry collision cylinder length=0.0532142958585139 radius=0.005; visual cylinder length=0.0532142958585139 radius=0.0035
- link arm31_pen_lead: geometry collision cylinder length=0.0532142958585139 radius=0.005; visual cylinder length=0.0532142958585139 radius=0.0035
- link arm71_pen_lead: geometry collision cylinder length=0.0532142958585139 radius=0.005; visual cylinder length=0.0532142958585139 radius=0.0035
- link arm97_pen_lead: geometry collision cylinder length=0.0532142958585139 radius=0.005; visual cylinder length=0.0532142958585139 radius=0.0035
Joints:
- joint arm13_pen_tip_weld: origin xyz=0.11 0.0 0.11 -> xyz=0.0588421 0.0 0.0588421
- joint arm17_pen_tip_weld: origin xyz=0.11 0.0 0.11 -> xyz=0.0588421 0.0 0.0588421
- joint arm2_pen_tip_weld: origin xyz=0.11 0.0 0.11 -> xyz=0.0588421 0.0 0.0588421
- joint arm31_pen_tip_weld: origin xyz=0.11 0.0 0.11 -> xyz=0.0588421 0.0 0.0588421
- joint arm71_pen_tip_weld: origin xyz=0.11 0.0 0.11 -> xyz=0.0588421 0.0 0.0588421
- joint arm97_pen_tip_weld: origin xyz=0.11 0.0 0.11 -> xyz=0.0588421 0.0 0.0588421

File: assets/system_model/installation_capsules.urdf (robot description, URDF)
Before this commit: robot aris_system_model_capsule, 186 links, 185 joints
Links:
- link arm13_pen_lead: geometry collision cylinder length=0.0532142958585139 radius=0.005; visual cylinder length=0.0532142958585139 radius=0.0035
- link arm17_pen_lead: geometry collision cylinder length=0.0532142958585139 radius=0.005; visual cylinder length=0.0532142958585139 radius=0.0035
- link arm2_pen_lead: geometry collision cylinder length=0.0532142958585139 radius=0.005; visual cylinder length=0.0532142958585139 radius=0.0035
- link arm31_pen_lead: geometry collision cylinder length=0.0532142958585139 radius=0.005; visual cylinder length=0.0532142958585139 radius=0.0035
- link arm71_pen_lead: geometry collision cylinder length=0.0532142958585139 radius=0.005; visual cylinder length=0.0532142958585139 radius=0.0035
- link arm97_pen_lead: geometry collision cylinder length=0.0532142958585139 radius=0.005; visual cylinder length=0.0532142958585139 radius=0.0035
Joints:
- joint arm13_pen_tip_weld: origin xyz=0.11 0.0 0.11 -> xyz=0.0588421 0.0 0.0588421
- joint arm17_pen_tip_weld: origin xyz=0.11 0.0 0.11 -> xyz=0.0588421 0.0 0.0588421
- joint arm2_pen_tip_weld: origin xyz=0.11 0.0 0.11 -> xyz=0.0588421 0.0 0.0588421
- joint arm31_pen_tip_weld: origin xyz=0.11 0.0 0.11 -> xyz=0.0588421 0.0 0.0588421
- joint arm71_pen_tip_weld: origin xyz=0.11 0.0 0.11 -> xyz=0.0588421 0.0 0.0588421
- joint arm97_pen_tip_weld: origin xyz=0.11 0.0 0.11 -> xyz=0.0588421 0.0 0.0588421

File: assets/system_model/installation_fatfingers.urdf (robot description, URDF)
Before this commit: robot aris_system_model_fatfingers, 186 links, 185 joints
Links:
- link arm13_pen_lead: geometry collision cylinder length=0.0532142958585139 radius=0.005; visual cylinder length=0.0532142958585139 radius=0.0035
- link arm17_pen_lead: geometry collision cylinder length=0.0532142958585139 radius=0.005; visual cylinder length=0.0532142958585139 radius=0.0035
- link arm2_pen_lead: geometry collision cylinder length=0.0532142958585139 radius=0.005; visual cylinder length=0.0532142958585139 radius=0.0035
- link arm31_pen_lead: geometry collision cylinder length=0.0532142958585139 radius=0.005; visual cylinder length=0.0532142958585139 radius=0.0035
- link arm71_pen_lead: geometry collision cylinder length=0.0532142958585139 radius=0.005; visual cylinder length=0.0532142958585139 radius=0.0035
- link arm97_pen_lead: geometry collision cylinder length=0.0532142958585139 radius=0.005; visual cylinder length=0.0532142958585139 radius=0.0035
Joints:
- joint arm13_pen_tip_weld: origin xyz=0.11 0.0 0.11 -> xyz=0.0588421 0.0 0.0588421
- joint arm17_pen_tip_weld: origin xyz=0.11 0.0 0.11 -> xyz=0.0588421 0.0 0.0588421
- joint arm2_pen_tip_weld: origin xyz=0.11 0.0 0.11 -> xyz=0.0588421 0.0 0.0588421
- joint arm31_pen_tip_weld: origin xyz=0.11 0.0 0.11 -> xyz=0.0588421 0.0 0.0588421
- joint arm71_pen_tip_weld: origin xyz=0.11 0.0 0.11 -> xyz=0.0588421 0.0 0.0588421
- joint arm97_pen_tip_weld: origin xyz=0.11 0.0 0.11 -> xyz=0.0588421 0.0 0.0588421
