Commit message: The holder was clamped in the middle of a 90 mm blade, and the photograph has it at the end
Pete, on the first render: "you need to move the pen to the front of the
aluminum extension … you essentially need to slide it forward in x by a few cm
so the gripping point is at the tip of the finger extension."

He is right, and the reason the model had it wrong is worth naming.  The Fat
finger's contact plate is 90 mm long and runs link x -9.000 .. +79.500 — the
90 mm is ACROSS the hand, not down the finger — and the only feature on it
that looks like it locates anything is the 6.000 mm hole on the finger
centreline.  It does not locate anything: 7d(a) says so in as many words, it
is an insert hole for a fingertip nobody fitted.  The post went on the
centreline anyway, and every render since has shown 66.5 mm of aluminium
hanging past the tool that the photograph does not show.

Clamped at the far end instead, a 26 mm post with its OUTER FACE FLUSH with
the plate's own far edge has its axis at 79.500 - 13.000 = 66.500 mm.  That is
`PENHOLDER22["grip_hand_x"]`, USER-SPECIFIED 2026-09-04, and the sign is not a
detail: both blades reach the same way in the hand (one part, mirrored) and
the bore leans the same way, so the tool is cantilevered the way the photo
shows.  Clamped at the far end with the pen leaning back over the wrist would
be a different and much worse tool.

NOTHING INSIDE THE HOLDER MOVES.  Sliding the grip along hand x translates the
whole assembly and nothing else: the bore still leans 45.00 deg, the grip is
still 30.001 mm from the cap's outer face and 55.099 mm from the tail face,
the graphite past the cap is the same 53.214 mm, and the grip HEIGHT and the
post-between-the-plates seating are untouched.  Every length in 7e's table
except the tip is a length along the holder, which is why they all survive.

THE TIP, AND ONE WORD IN THE VOCABULARY.

    grip centre       (0, 0, 0.1034)  ->  (0.066500, 0, 0.1034)
    PEN_EXT_HOLDER    0.0588421       ->  0.0588421      (unchanged: the tip
                                                          is still 50.000 mm
                                                          below the plates)
    PEN_LAT_HOLDER    0.0588421       ->  0.1253421      = grip_hand_x +
                                                          PEN_EXT_HOLDER*tan45
    tip, panda_hand   (0.0588, 0, 0.1622) -> (0.1253421, 0, 0.1622421)

`PEN_LEAN_HOLDER` is still 45 deg and now says which 45 deg it is: the BORE's
lean, measured AT THE GRIP, which is what a protractor on the real barrel
reads.  It stopped being the angle of the TCP -> tip ray the moment the grip
left the TCP — that ray leans 64.85 deg — and `penholder22_T_hand` aims the
bore at the GRIP -> tip ray instead.  Both generators used to rebuild the
graphite from `arctan2(pen_lat, pen_ext)` and would now have drawn 53 mm of it
20 deg off the barrel; `rig_final.penholder22_lead` owns that arithmetic in
one place and a test pins it.

AND THIS WITHDRAWS AN ARGUMENT I MADE YESTERDAY.  With the grip on the
centreline the gripper's own casing ruled out any lean under 35.17 deg, and
that was the reason given for 45.  At the far-end placement it is not true:

                              centreline        far end
    housing vs hand, 23 deg    -11.90 mm       +13.84 mm
    housing vs hand, 45 deg     +6.15 mm        +7.78 mm
    cap, 45 deg                +40.44 mm       +81.87 mm
    the 72.5 mm tail, 45 deg   +18.36 mm       -24.32 mm

23 deg now clears the casing BETTER than 45 does.  So the lean is 45 because
it is the user's standing rule and the incumbent, not because the hardware
forces it, and 7e, DECISIONS.md, `system_model.OPEN_QUESTIONS`, README and
LAYOUT_STUDY all say so where they said the opposite.  Per the user the casing
does not constrain the model at all for now — "the pen's simulated length is a
random number at this point so it does not matter if it intersects with the
gripper casing" — so the -24.32 mm, 24 mm of pencil tail drawn through the
casting, is REPORTED and not designed around.  The barrel itself is clear.

REGENERATED, and this time the holder meshes DO move: they carry the placement
baked in, so `assets/system_model/meshes/penholder/*` and
`assets/proposed_rig/meshes/*` are re-baked along with four URDFs, the
manifest and MESH_SOURCES.  `check_system_model.py` ALL PASS, worst pen tip
4.555e-12 m over 25 configs x 6 arms, with two new assertions: the bore points
along the GRIP -> tip ray, and the grip centre lands where a 26 mm post is
flush with the plate's far edge.  `check_proposed_rig_urdf.py` ALL PASS,
9.365e-10 m.

The two close-up cameras aim at the grip now instead of down the wrist
centreline — a subject 66.5 mm off axis was at the edge of its own frame.
`out/system_model_fatfingers_{holder,holder_side,photo}.png` and the seven
stock-finger views are re-rendered; `photo` is the one to hold against the
photograph.

Tests: `test_system_model`, `test_proposed_rig_urdf`, `test_lateral`,
`test_gates`, `test_mounts`, `test_final_rig`, `test_selfcoll` — 153 passed,
1 skipped.  Four pinned tests moved from the TCP -> tip ray to the GRIP -> tip
ray with the reason in their docstrings.

NOT TOUCHED, AND IT IS NOW STALE AGAIN: `layout.Q_PARK_PROPOSED` and
`tests/test_layout.py` belong to the park re-search another agent committed in
0120980, and this commit invalidates it a second time — its own message says
"and then the grip point moved again".  Measured before leaving it alone: all
six of those poses still PASS `validate.check_pose` at the new tool, the fleet
holds 250 mm against an 80 mm gate, and the tip HEIGHTS are untouched (they
depend on `PEN_EXT_HOLDER`, which did not move) — what moved is each tip's
in-plane position, by 66.5 mm.  So they are safe and they are no longer the
search's own output; three assertions in `tests/test_layout.py` are red until
that search is re-run.

Co-Authored-By: Claude Opus 5 <noreply@anthropic.com>
Claude-Session: https://claude.ai/code/session_01TYL3Cueh7sskNU8Uz21h7x

File: assets/proposed_rig/installation.urdf (robot description, URDF)
Before this commit: robot aris_proposed_rig, 123 links, 122 joints
Links:
- link arm13_pen_bracket: geometry collision cylinder length=0.1253421 radius=0.05
- link arm17_pen_bracket: geometry collision cylinder length=0.1253421 radius=0.05
- link arm2_pen_bracket: geometry collision cylinder length=0.1253421 radius=0.05
- link arm31_pen_bracket: geometry collision cylinder length=0.1253421 radius=0.05
- link arm71_pen_bracket: geometry collision cylinder length=0.1253421 radius=0.05
- link arm97_pen_bracket: geometry collision cylinder length=0.1253421 radius=0.05
Joints:
- joint arm13_pen_body_weld: origin xyz=0.0588421 0 0 -> xyz=0.1253421 0 0
- joint arm17_pen_body_weld: origin xyz=0.0588421 0 0 -> xyz=0.1253421 0 0
- joint arm2_pen_body_weld: origin xyz=0.0588421 0 0 -> xyz=0.1253421 0 0
- joint arm31_pen_body_weld: origin xyz=0.0588421 0 0 -> xyz=0.1253421 0 0
- joint arm71_pen_body_weld: origin xyz=0.0588421 0 0 -> xyz=0.1253421 0 0
- joint arm97_pen_body_weld: origin xyz=0.0588421 0 0 -> xyz=0.1253421 0 0

File: assets/system_model/installation.urdf (robot description, URDF)
Before this commit: robot aris_system_model, 186 links, 185 joints
Joints:
- joint arm13_pen_tip_weld: origin xyz=0.0588421 0.0 0.0588421 -> xyz=0.1253421 0.0 0.0588421
- joint arm17_pen_tip_weld: origin xyz=0.0588421 0.0 0.0588421 -> xyz=0.1253421 0.0 0.0588421
- joint arm2_pen_tip_weld: origin xyz=0.0588421 0.0 0.0588421 -> xyz=0.1253421 0.0 0.0588421
- joint arm31_pen_tip_weld: origin xyz=0.0588421 0.0 0.0588421 -> xyz=0.1253421 0.0 0.0588421
- joint arm71_pen_tip_weld: origin xyz=0.0588421 0.0 0.0588421 -> xyz=0.1253421 0.0 0.0588421
- joint arm97_pen_tip_weld: origin xyz=0.0588421 0.0 0.0588421 -> xyz=0.1253421 0.0 0.0588421

File: assets/system_model/installation_capsules.urdf (robot description, URDF)
Before this commit: robot aris_system_model_capsule, 186 links, 185 joints
Joints:
- joint arm13_pen_tip_weld: origin xyz=0.0588421 0.0 0.0588421 -> xyz=0.1253421 0.0 0.0588421
- joint arm17_pen_tip_weld: origin xyz=0.0588421 0.0 0.0588421 -> xyz=0.1253421 0.0 0.0588421
- joint arm2_pen_tip_weld: origin xyz=0.0588421 0.0 0.0588421 -> xyz=0.1253421 0.0 0.0588421
- joint arm31_pen_tip_weld: origin xyz=0.0588421 0.0 0.0588421 -> xyz=0.1253421 0.0 0.0588421
- joint arm71_pen_tip_weld: origin xyz=0.0588421 0.0 0.0588421 -> xyz=0.1253421 0.0 0.0588421
- joint arm97_pen_tip_weld: origin xyz=0.0588421 0.0 0.0588421 -> xyz=0.1253421 0.0 0.0588421

File: assets/system_model/installation_fatfingers.urdf (robot description, URDF)
Before this commit: robot aris_system_model_fatfingers, 186 links, 185 joints
Joints:
- joint arm13_pen_tip_weld: origin xyz=0.0588421 0.0 0.0588421 -> xyz=0.1253421 0.0 0.0588421
- joint arm17_pen_tip_weld: origin xyz=0.0588421 0.0 0.0588421 -> xyz=0.1253421 0.0 0.0588421
- joint arm2_pen_tip_weld: origin xyz=0.0588421 0.0 0.0588421 -> xyz=0.1253421 0.0 0.0588421
- joint arm31_pen_tip_weld: origin xyz=0.0588421 0.0 0.0588421 -> xyz=0.1253421 0.0 0.0588421
- joint arm71_pen_tip_weld: origin xyz=0.0588421 0.0 0.0588421 -> xyz=0.1253421 0.0 0.0588421
- joint arm97_pen_tip_weld: origin xyz=0.0588421 0.0 0.0588421 -> xyz=0.1253421 0.0 0.0588421

Commit message: The square block is flush with the blades at 23 degrees and at no other lean, which is the CAD's own number
Two corrections off the side view down the jaw axis, and the second one is a
measurement wearing plain clothes.

"IN THE PICTURE THE SQUARE PART OF THE HOLDER IS FLUSH WITH THE METAL PART, so
the entire pen-holder plastic bit that is being pinched is about 20 degrees
more upright."  That is not a preference, it is a protractor.  The mount post
is a 26 mm square whose four flats are clocked `PENHOLDER22["post_clock"]` =
23.00 deg about the post axis relative to the bore — measured off the STL here
rather than taken on trust: the four large flats' normals sit at -113.00 /
-23.00 / +67.00 / +157.00 deg from the housing's own +X, which IS the bore.
The post axis is hand y, so those normals live in the hand's x-z plane, and:

    bore 45 deg -> flat normals at -158 / -68 / +22 / +112 off hand z  (askew)
    bore 23 deg -> flat normals at -180 /  -90 /   0 /  +90            (SQUARE)

The block is flush with the blades' plate faces and edges at 23 deg and at no
other lean, and the 22 deg it was out is exactly the "about 20 degrees more
upright" Pete asked for.  `PEN_LEAN_HOLDER` = 23 deg.

SO THE 22-DEGREE RED FLAG CLOSES, IN THE CAD'S FAVOUR.  It has been the
biggest open question in docs/SYSTEM_MODEL.md since 2026-08-25: the housing's
own flats said 23, the model drew 45, and no mechanism could carry the
difference — not a cradle, not the fingertip sockets, not the Fat blade.  It
turns out none was needed.  The 45 was a planner assumption that nothing ever
supported, propped up for one day (2026-09-03) by a casing argument that was
itself withdrawn on 2026-09-04 when the grip moved to the plates' far end.
`extract_penholder22_meshes.py` has printed that disagreement on every run for
a fortnight.  It now prints -0.00 deg.

AND THE TIP COMES OFF THE HOLDER RATHER THAN OFF THE BLADES.  "Shorten the
shaft of the pen … I think it only juts out 3-4 cm max", then, with the
orientation confirmed against the real gripper ("looks great now"), about
2 cm.  So `PEN_GRAPHITE_HOLDER` = 20 mm past the cap's outer face is an INPUT
now, and the whole transform is one line:

    grip  = (0.066500, 0, 0.1034)          the far end of the Fat blades
    u     = (sin 23, 0, cos 23)          = (0.390731, 0, 0.920505)
    tip   = grip + (30.001 + 20.000) mm * u
          = (0.0860369, 0, 0.1494262)
    PEN_EXT_HOLDER = 0.0460262    PEN_LAT_HOLDER = 0.0860369

THIS SUPERSEDES — and this time contradicts — the "tip 50 mm below the bottom
edge of the blades" rule of 2026-09-03.  The derived tip sits 37.18 mm below
that edge, not 50.  Said plainly rather than smoothed over: the blades' edge
was a plausible datum for a tip nobody had measured, and the holder is a
better one, because the protrusion is the thing a person can see and adjust.
One corroboration that is not an argument but is worth writing down: 20 mm of
graphite + the 85.100 mm barrel + the assembly's 72.514 mm tail is a 177.6 mm
stick, and a Cretacolor Monolith is 175 mm.  Every earlier tip asked for a
stick nobody sells.

The grip centre does not move (0.066500, 0, 0.1034), the housing's internals
do not move, and `PEN_LEAN_HOLDER` still means what it started meaning on
2026-09-04: the BORE's lean measured AT THE GRIP, which is what a protractor
on the real barrel reads.  The TCP -> tip ray is 61.86 deg and is a different
line; `penholder22_T_hand` aims the bore at the grip -> tip ray and
`penholder22_lead` owns the graphite, so neither generator can drift.

CASING CLEARANCE STAYS IRRELEVANT BY INSTRUCTION and is reported only: at this
lean the housing clears the manufacturer's hand shell by +13.84 mm, the cap by
+59.90, and the 72.5 mm pencil tail runs -10.61 mm into it.  None of those
numbers moved with the graphite; only the tip did.

REGENERATED: the holder meshes carry the placement baked in, so both asset
trees' `penholder22_*_hand.obj` are re-baked along with four URDFs, the
manifest and MESH_SOURCES.  `check_system_model.py` ALL PASS, worst pen tip
4.524e-12 m over 25 configs x 6 arms, including the bore-along-grip->tip
assertion and the grip-at-the-plate-end assertion.
`check_proposed_rig_urdf.py` ALL PASS.

NEW RENDER, `--views holder_jaw`: straight down the JAW axis, aimed at the
holder's own middle, up = -z_hand.  The bore's lean and the graphite's
protrusion both lie IN the image plane there, so neither is foreshortened —
which is what makes it the shot to hold against a photograph, and it is the
view these two corrections came out of.  `holder_side` looks down hand x and
shows the V of the blades; this one looks down hand y and shows the ANGLE.

Tests: test_system_model, test_proposed_rig_urdf, test_lateral, test_gates,
test_mounts, test_final_rig, test_selfcoll — 153 passed, 1 skipped.  The
pinned lean, graphite and tip-below-blades assertions moved with the reason in
their docstrings, and the 23 deg one is pinned against `post_clock` rather
than against a literal, so the test says WHY 23 rather than that it is 23.

`layout.Q_PARK_PROPOSED` and `tests/test_layout.py` are untouched: they belong
to the park re-search that follows from this commit.

Co-Authored-By: Claude Opus 5 <noreply@anthropic.com>
Claude-Session: https://claude.ai/code/session_01TYL3Cueh7sskNU8Uz21h7x

File: assets/proposed_rig/installation.urdf (robot description, URDF)
Before this commit: robot aris_proposed_rig, 123 links, 122 joints
Links:
- link arm13_pen_body: geometry collision cylinder length=0.0460262 radius=0.05
- link arm13_pen_bracket: geometry collision cylinder length=0.0860369 radius=0.05
- link arm13_pen_lead: geometry collision cylinder length=0.020000015 radius=0.005; visual cylinder length=0.020000015 radius=0.0035
- link arm17_pen_body: geometry collision cylinder length=0.0460262 radius=0.05
- link arm17_pen_bracket: geometry collision cylinder length=0.0860369 radius=0.05
- link arm17_pen_lead: geometry collision cylinder length=0.020000015 radius=0.005; visual cylinder length=0.020000015 radius=0.0035
- link arm2_pen_body: geometry collision cylinder length=0.0460262 radius=0.05
- link arm2_pen_bracket: geometry collision cylinder length=0.0860369 radius=0.05
- link arm2_pen_lead: geometry collision cylinder length=0.020000015 radius=0.005; visual cylinder length=0.020000015 radius=0.0035
- link arm31_pen_body: geometry collision cylinder length=0.0460262 radius=0.05
- link arm31_pen_bracket: geometry collision cylinder length=0.0860369 radius=0.05
- link arm31_pen_lead: geometry collision cylinder length=0.020000015 radius=0.005; visual cylinder length=0.020000015 radius=0.0035
- link arm71_pen_body: geometry collision cylinder length=0.0460262 radius=0.05
- link arm71_pen_bracket: geometry collision cylinder length=0.0860369 radius=0.05
- link arm71_pen_lead: geometry collision cylinder length=0.020000015 radius=0.005; visual cylinder length=0.020000015 radius=0.0035
- link arm97_pen_body: geometry collision cylinder length=0.0460262 radius=0.05
- link arm97_pen_bracket: geometry collision cylinder length=0.0860369 radius=0.05
- link arm97_pen_lead: geometry collision cylinder length=0.020000015 radius=0.005; visual cylinder length=0.020000015 radius=0.0035
Joints:
- joint arm13_pen_body_weld: origin xyz=0.1253421 0 0 -> xyz=0.0860369 0 0
- joint arm13_pen_tip_weld: origin xyz=0 0 0.0588421 -> xyz=0 0 0.0460262
- joint arm17_pen_body_weld: origin xyz=0.1253421 0 0 -> xyz=0.0860369 0 0
- joint arm17_pen_tip_weld: origin xyz=0 0 0.0588421 -> xyz=0 0 0.0460262
- joint arm2_pen_body_weld: origin xyz=0.1253421 0 0 -> xyz=0.0860369 0 0
- joint arm2_pen_tip_weld: origin xyz=0 0 0.0588421 -> xyz=0 0 0.0460262
- joint arm31_pen_body_weld: origin xyz=0.1253421 0 0 -> xyz=0.0860369 0 0
- joint arm31_pen_tip_weld: origin xyz=0 0 0.0588421 -> xyz=0 0 0.0460262
- joint arm71_pen_body_weld: origin xyz=0.1253421 0 0 -> xyz=0.0860369 0 0
- joint arm71_pen_tip_weld: origin xyz=0 0 0.0588421 -> xyz=0 0 0.0460262
- joint arm97_pen_body_weld: origin xyz=0.1253421 0 0 -> xyz=0.0860369 0 0
- joint arm97_pen_tip_weld: origin xyz=0 0 0.0588421 -> xyz=0 0 0.0460262

File: assets/system_model/installation.urdf (robot description, URDF)
Before this commit: robot aris_system_model, 186 links, 185 joints
Links:
- link arm13_pen_lead: geometry collision cylinder length=0.020000015470188197 radius=0.005; visual cylinder length=0.020000015470188197 radius=0.0035
- link arm17_pen_lead: geometry collision cylinder length=0.020000015470188197 radius=0.005; visual cylinder length=0.020000015470188197 radius=0.0035
- link arm2_pen_lead: geometry collision cylinder length=0.020000015470188197 radius=0.005; visual cylinder length=0.020000015470188197 radius=0.0035
- link arm31_pen_lead: geometry collision cylinder length=0.020000015470188197 radius=0.005; visual cylinder length=0.020000015470188197 radius=0.0035
- link arm71_pen_lead: geometry collision cylinder length=0.020000015470188197 radius=0.005; visual cylinder length=0.020000015470188197 radius=0.0035
- link arm97_pen_lead: geometry collision cylinder length=0.020000015470188197 radius=0.005; visual cylinder length=0.020000015470188197 radius=0.0035
Joints:
- joint arm13_pen_tip_weld: origin xyz=0.1253421 0.0 0.0588421 -> xyz=0.0860369 0.0 0.0460262
- joint arm17_pen_tip_weld: origin xyz=0.1253421 0.0 0.0588421 -> xyz=0.0860369 0.0 0.0460262
- joint arm2_pen_tip_weld: origin xyz=0.1253421 0.0 0.0588421 -> xyz=0.0860369 0.0 0.0460262
- joint arm31_pen_tip_weld: origin xyz=0.1253421 0.0 0.0588421 -> xyz=0.0860369 0.0 0.0460262
- joint arm71_pen_tip_weld: origin xyz=0.1253421 0.0 0.0588421 -> xyz=0.0860369 0.0 0.0460262
- joint arm97_pen_tip_weld: origin xyz=0.1253421 0.0 0.0588421 -> xyz=0.0860369 0.0 0.0460262

File: assets/system_model/installation_capsules.urdf (robot description, URDF)
Before this commit: robot aris_system_model_capsule, 186 links, 185 joints
Links:
- link arm13_pen_lead: geometry collision cylinder length=0.020000015470188197 radius=0.005; visual cylinder length=0.020000015470188197 radius=0.0035
- link arm17_pen_lead: geometry collision cylinder length=0.020000015470188197 radius=0.005; visual cylinder length=0.020000015470188197 radius=0.0035
- link arm2_pen_lead: geometry collision cylinder length=0.020000015470188197 radius=0.005; visual cylinder length=0.020000015470188197 radius=0.0035
- link arm31_pen_lead: geometry collision cylinder length=0.020000015470188197 radius=0.005; visual cylinder length=0.020000015470188197 radius=0.0035
- link arm71_pen_lead: geometry collision cylinder length=0.020000015470188197 radius=0.005; visual cylinder length=0.020000015470188197 radius=0.0035
- link arm97_pen_lead: geometry collision cylinder length=0.020000015470188197 radius=0.005; visual cylinder length=0.020000015470188197 radius=0.0035
Joints:
- joint arm13_pen_tip_weld: origin xyz=0.1253421 0.0 0.0588421 -> xyz=0.0860369 0.0 0.0460262
- joint arm17_pen_tip_weld: origin xyz=0.1253421 0.0 0.0588421 -> xyz=0.0860369 0.0 0.0460262
- joint arm2_pen_tip_weld: origin xyz=0.1253421 0.0 0.0588421 -> xyz=0.0860369 0.0 0.0460262
- joint arm31_pen_tip_weld: origin xyz=0.1253421 0.0 0.0588421 -> xyz=0.0860369 0.0 0.0460262
- joint arm71_pen_tip_weld: origin xyz=0.1253421 0.0 0.0588421 -> xyz=0.0860369 0.0 0.0460262
- joint arm97_pen_tip_weld: origin xyz=0.1253421 0.0 0.0588421 -> xyz=0.0860369 0.0 0.0460262

File: assets/system_model/installation_fatfingers.urdf (robot description, URDF)
Before this commit: robot aris_system_model_fatfingers, 186 links, 185 joints
Links:
- link arm13_pen_lead: geometry collision cylinder length=0.020000015470188197 radius=0.005; visual cylinder length=0.020000015470188197 radius=0.0035
- link arm17_pen_lead: geometry collision cylinder length=0.020000015470188197 radius=0.005; visual cylinder length=0.020000015470188197 radius=0.0035
- link arm2_pen_lead: geometry collision cylinder length=0.020000015470188197 radius=0.005; visual cylinder length=0.020000015470188197 radius=0.0035
- link arm31_pen_lead: geometry collision cylinder length=0.020000015470188197 radius=0.005; visual cylinder length=0.020000015470188197 radius=0.0035
- link arm71_pen_lead: geometry collision cylinder length=0.020000015470188197 radius=0.005; visual cylinder length=0.020000015470188197 radius=0.0035
- link arm97_pen_lead: geometry collision cylinder length=0.020000015470188197 radius=0.005; visual cylinder length=0.020000015470188197 radius=0.0035
Joints:
- joint arm13_pen_tip_weld: origin xyz=0.1253421 0.0 0.0588421 -> xyz=0.0860369 0.0 0.0460262
- joint arm17_pen_tip_weld: origin xyz=0.1253421 0.0 0.0588421 -> xyz=0.0860369 0.0 0.0460262
- joint arm2_pen_tip_weld: origin xyz=0.1253421 0.0 0.0588421 -> xyz=0.0860369 0.0 0.0460262
- joint arm31_pen_tip_weld: origin xyz=0.1253421 0.0 0.0588421 -> xyz=0.0860369 0.0 0.0460262
- joint arm71_pen_tip_weld: origin xyz=0.1253421 0.0 0.0588421 -> xyz=0.0860369 0.0 0.0460262
- joint arm97_pen_tip_weld: origin xyz=0.1253421 0.0 0.0588421 -> xyz=0.0860369 0.0 0.0460262
