Commit message: The assembly file this holder was said not to have was inside the zip, two levels down
`Pen holder cad(1).zip` nests `Natural hold assembly - closed.zip`, and that
holds `Natural hold assembly - closed.SLDASM`: the complete 10-deg build,
seven components, mated, with two FR3 fingertips in it.  The files are the
SolidWorks 2024/25 container — nibble-swapped stream names, raw-deflate
payloads — so the component transforms come out of
`swXmlContents/COMPINSTANCETREE` and the per-part boxes out of
`Contents/DisplayLists`, both cross-checked against the STLs of the parts the
2026.08.19 delivery does ship.

That assembly is the same architecture as this one part-for-part, so it fixes
the axial ORDER eight loose STLs cannot: nose shoulder -> spring -> [shim] ->
sleeve (clutch inside it) -> cap shoulder.  Every interface is then re-measured
on this delivery's own parts: a 21.0 face lands on the nose chamfer at 3.340,
the cap is a threaded COLLAR whose 16.00 shoulder at 83.115 is the back stop,
79.775 of space less the 40.100 sleeve squeezes the 50.81 spring to 39.675 —
11.135 mm of preload with 11.175 left before coil bind.  The two spacers are a
SHIM SET, not a stack: one of {none, 5, 10} sets that preload, and both at once
asks 26.3 mm of a spring with 22.3 to solid.  The clutch is a split collet and
the sleeve's 15.030 -> 16.290 bore is its taper; the tapers match to
0.00003 mm/mm, and the 13.0 land they end in is the bench extractor's guide,
which is why that 12.0 x 40 pusher rod is the shape it is.

The stack is drawn, VISUAL ONLY, and the collision hull is untouched: all five
bodies live inside the 21.148 bore, and the generator now refuses to write a
URDF unless `penholder22_internals_escape` measures 0.0 for the complete
assembly.  It does, for all three shim settings.

And the fingers moved.  The post is 50 mm long with a 7.000 socket in each end,
so the faces the fingertips seat on are 36.000 apart — the assembly puts them
at 36.0008.  `FINGER_FIX` was 0.0285, which is the fingertip's BACK face:
50 + 2 x 3.5 added the tip left OUTSIDE the socket instead of subtracting the
7 mm inside it, and 57 mm is 7 mm wider than the post is long.  At 0.018 the
URDF's finger lands where the assembly puts it in all three axes.

Co-Authored-By: Claude Opus 5 <noreply@anthropic.com>
Claude-Session: https://claude.ai/code/session_01TYL3Cueh7sskNU8Uz21h7x

File: assets/system_model/installation.urdf (robot description, URDF)
Before this commit: robot aris_system_model, 186 links, 185 joints
Links:
- link arm13_pen_holder: geometry collision cylinder length=0.01150000000000001 radius=0.0181; collision cylinder length=0.035 radius=0.0136
- link arm17_pen_holder: geometry collision cylinder length=0.01150000000000001 radius=0.0181; collision cylinder length=0.035 radius=0.0136
- link arm2_pen_holder: geometry collision cylinder length=0.01150000000000001 radius=0.0181; collision cylinder length=0.035 radius=0.0136
- link arm31_pen_holder: geometry collision cylinder length=0.01150000000000001 radius=0.0181; collision cylinder length=0.035 radius=0.0136
- link arm71_pen_holder: geometry collision cylinder length=0.01150000000000001 radius=0.0181; collision cylinder length=0.035 radius=0.0136
- link arm97_pen_holder: geometry collision cylinder length=0.01150000000000001 radius=0.0181; collision cylinder length=0.035 radius=0.0136
Joints:
- joint arm13_panda_finger_joint1: origin xyz=0.0 0.0285 0.0584 rpy=0 0 0 -> xyz=0.0 0.018 0.0584 rpy=0 0 0
- joint arm13_panda_finger_joint2: origin xyz=0.0 -0.0285 0.0584 rpy=0 0 0 -> xyz=0.0 -0.018 0.0584 rpy=0 0 0
- joint arm17_panda_finger_joint1: origin xyz=0.0 0.0285 0.0584 rpy=0 0 0 -> xyz=0.0 0.018 0.0584 rpy=0 0 0
- joint arm17_panda_finger_joint2: origin xyz=0.0 -0.0285 0.0584 rpy=0 0 0 -> xyz=0.0 -0.018 0.0584 rpy=0 0 0
- joint arm2_panda_finger_joint1: origin xyz=0.0 0.0285 0.0584 rpy=0 0 0 -> xyz=0.0 0.018 0.0584 rpy=0 0 0
- joint arm2_panda_finger_joint2: origin xyz=0.0 -0.0285 0.0584 rpy=0 0 0 -> xyz=0.0 -0.018 0.0584 rpy=0 0 0
- joint arm31_panda_finger_joint1: origin xyz=0.0 0.0285 0.0584 rpy=0 0 0 -> xyz=0.0 0.018 0.0584 rpy=0 0 0
- joint arm31_panda_finger_joint2: origin xyz=0.0 -0.0285 0.0584 rpy=0 0 0 -> xyz=0.0 -0.018 0.0584 rpy=0 0 0
- joint arm71_panda_finger_joint1: origin xyz=0.0 0.0285 0.0584 rpy=0 0 0 -> xyz=0.0 0.018 0.0584 rpy=0 0 0
- joint arm71_panda_finger_joint2: origin xyz=0.0 -0.0285 0.0584 rpy=0 0 0 -> xyz=0.0 -0.018 0.0584 rpy=0 0 0
- joint arm97_panda_finger_joint1: origin xyz=0.0 0.0285 0.0584 rpy=0 0 0 -> xyz=0.0 0.018 0.0584 rpy=0 0 0
- joint arm97_panda_finger_joint2: origin xyz=0.0 -0.0285 0.0584 rpy=0 0 0 -> xyz=0.0 -0.018 0.0584 rpy=0 0 0

File: assets/system_model/installation_capsules.urdf (robot description, URDF)
Before this commit: robot aris_system_model_capsule, 186 links, 185 joints
Links:
- link arm13_pen_holder: geometry collision cylinder length=0.01150000000000001 radius=0.0181; collision cylinder length=0.035 radius=0.0136
- link arm17_pen_holder: geometry collision cylinder length=0.01150000000000001 radius=0.0181; collision cylinder length=0.035 radius=0.0136
- link arm2_pen_holder: geometry collision cylinder length=0.01150000000000001 radius=0.0181; collision cylinder length=0.035 radius=0.0136
- link arm31_pen_holder: geometry collision cylinder length=0.01150000000000001 radius=0.0181; collision cylinder length=0.035 radius=0.0136
- link arm71_pen_holder: geometry collision cylinder length=0.01150000000000001 radius=0.0181; collision cylinder length=0.035 radius=0.0136
- link arm97_pen_holder: geometry collision cylinder length=0.01150000000000001 radius=0.0181; collision cylinder length=0.035 radius=0.0136
Joints:
- joint arm13_panda_finger_joint1: origin xyz=0.0 0.0285 0.0584 rpy=0 0 0 -> xyz=0.0 0.018 0.0584 rpy=0 0 0
- joint arm13_panda_finger_joint2: origin xyz=0.0 -0.0285 0.0584 rpy=0 0 0 -> xyz=0.0 -0.018 0.0584 rpy=0 0 0
- joint arm17_panda_finger_joint1: origin xyz=0.0 0.0285 0.0584 rpy=0 0 0 -> xyz=0.0 0.018 0.0584 rpy=0 0 0
- joint arm17_panda_finger_joint2: origin xyz=0.0 -0.0285 0.0584 rpy=0 0 0 -> xyz=0.0 -0.018 0.0584 rpy=0 0 0
- joint arm2_panda_finger_joint1: origin xyz=0.0 0.0285 0.0584 rpy=0 0 0 -> xyz=0.0 0.018 0.0584 rpy=0 0 0
- joint arm2_panda_finger_joint2: origin xyz=0.0 -0.0285 0.0584 rpy=0 0 0 -> xyz=0.0 -0.018 0.0584 rpy=0 0 0
- joint arm31_panda_finger_joint1: origin xyz=0.0 0.0285 0.0584 rpy=0 0 0 -> xyz=0.0 0.018 0.0584 rpy=0 0 0
- joint arm31_panda_finger_joint2: origin xyz=0.0 -0.0285 0.0584 rpy=0 0 0 -> xyz=0.0 -0.018 0.0584 rpy=0 0 0
- joint arm71_panda_finger_joint1: origin xyz=0.0 0.0285 0.0584 rpy=0 0 0 -> xyz=0.0 0.018 0.0584 rpy=0 0 0
- joint arm71_panda_finger_joint2: origin xyz=0.0 -0.0285 0.0584 rpy=0 0 0 -> xyz=0.0 -0.018 0.0584 rpy=0 0 0
- joint arm97_panda_finger_joint1: origin xyz=0.0 0.0285 0.0584 rpy=0 0 0 -> xyz=0.0 0.018 0.0584 rpy=0 0 0
- joint arm97_panda_finger_joint2: origin xyz=0.0 -0.0285 0.0584 rpy=0 0 0 -> xyz=0.0 -0.018 0.0584 rpy=0 0 0
