Commit message: A re-cert queue that measures against the bounding box of two boxes reports every escape above the plate 13 mm short
Four real errors, found by review.

THE RE-CERT NUMBERS WERE LOW.  `recert_escape_mm` merged the two envelope
boxes into one AABB, and they stack in z without sharing a footprint: the
plate is 226 x 190 and the column above it is 200 x 200.  A gusset 1.5 m up,
where only the column exists, was being scored against a 226-wide envelope.
54 of 60 bodies read 13 mm short and the queue's worst case said 172.55 where
it is 185.55.  Under-reporting is the wrong direction for a re-cert queue, and
the function's own docstring already said 38.15 for the clamp — it was written
against the right measure and the code was not it.  The bands are walked
separately now.  clamp 38.15, post to 122.05, gusset to 185.55, plate 25.06.

THE LEGS WERE 76.2 MM INSIDE THE RAILS THEY CARRY.  Drawn to the perimeter
rail's TOP instead of its underside, the way the drop posts already stop under
the runway.  `reconciliation()` published 1727.2 mm as a leg length and no
one can cut that; it is 1651.0.  The table is inset to the frame's inner span
for the same reason — drawn out to the outside it swallowed the legs' bottom
25 mm.  A new test intersects all 77 bodies pairwise and there is nothing left.

THE PLATE ROW CONTRADICTED THE ROW ABOVE IT.  One said the plate escapes by
25.06 mm in plan; the next said "the real one is inside it" and
`action="none"`.  The second is what a fabricator would act on.  Conservative
in thickness, out by 25.06 in plan, and re-cert either way.

THE DATUM DOCSTRING GOT ITS OWN ARITHMETIC WRONG, in the module whose whole
subject is a floor-versus-paper confusion: 2976.68 is the code datum's grid
UNDERSIDE above the FLOOR, not the top of the cage above the paper, which is
2416.2.  Both numbers, both datums, spelled out.

And the 7.34 mm the plate clearance was quoted at is the slot the DRAWING's
77.2 mm booms leave.  This model builds nominal 76.2 posts, so its slot is
241.4 and its clearance 7.79.  Both are carried; the test measures the posts
the model emits instead of reading the constant.

The tests that should have caught all of this are fixed too: the plate-nests
test read a constant, the re-cert test re-derived through the function it was
testing, the holder-envelope test never checked the cylinder AXIS (the
"coaxial with the bore" claim was unverified), and the shell test set-matched
where both fingers name one mesh.

39 tests.  Baseline confirmed at 345 passed / 9 skipped before any of this.

Co-Authored-By: Claude Opus 5 <noreply@anthropic.com>
Claude-Session: https://claude.ai/code/session_01TYL3Cueh7sskNU8Uz21h7x

File: assets/system_model/environment.urdf (robot description, URDF)
Before this commit: robot aris_system_model_env, 78 links, 77 joints
Links:
- link leg_BL: geometry collision box size=0.0762 0.0761999999999996 1.6509999999999998; visual box size=0.0762 0.0761999999999996 1.6509999999999998
- link leg_BR: geometry collision box size=0.07620000000000005 0.0761999999999996 1.6509999999999998; visual box size=0.07620000000000005 0.0761999999999996 1.6509999999999998
- link leg_FL: geometry collision box size=0.0762 0.0762 1.6509999999999998; visual box size=0.0762 0.0762 1.6509999999999998
- link leg_FR: geometry collision box size=0.07620000000000005 0.0762 1.6509999999999998; visual box size=0.07620000000000005 0.0762 1.6509999999999998
- link table: geometry collision box size=2.032 3.8592400000000002 0.6346799999999999; visual box size=2.032 3.8592400000000002 0.6346799999999999
Joints:
- joint leg_BL_weld: origin xyz=-0.1524 3.7830399999999997 0.83622 -> xyz=-0.1524 3.7830399999999997 0.7981199999999999
- joint leg_BR_weld: origin xyz=1.9558 3.7830399999999997 0.83622 -> xyz=1.9558 3.7830399999999997 0.7981199999999999
- joint leg_FL_weld: origin xyz=-0.1524 -0.1524 0.83622 -> xyz=-0.1524 -0.1524 0.7981199999999999
- joint leg_FR_weld: origin xyz=1.9558 -0.1524 0.83622 -> xyz=1.9558 -0.1524 0.7981199999999999
- joint table_weld: origin xyz=0.9017 1.8153199999999998 -0.31933999999999996 -> xyz=0.9017 1.81532 -0.31933999999999996

File: assets/system_model/installation.urdf (robot description, URDF)
Before this commit: robot aris_system_model, 186 links, 185 joints
Links:
- link leg_BL: geometry collision box size=0.0762 0.0761999999999996 1.6509999999999998; visual box size=0.0762 0.0761999999999996 1.6509999999999998
- link leg_BR: geometry collision box size=0.07620000000000005 0.0761999999999996 1.6509999999999998; visual box size=0.07620000000000005 0.0761999999999996 1.6509999999999998
- link leg_FL: geometry collision box size=0.0762 0.0762 1.6509999999999998; visual box size=0.0762 0.0762 1.6509999999999998
- link leg_FR: geometry collision box size=0.07620000000000005 0.0762 1.6509999999999998; visual box size=0.07620000000000005 0.0762 1.6509999999999998
- link table: geometry collision box size=2.032 3.8592400000000002 0.6346799999999999; visual box size=2.032 3.8592400000000002 0.6346799999999999
Joints:
- joint leg_BL_weld: origin xyz=-0.1524 3.7830399999999997 0.83622 -> xyz=-0.1524 3.7830399999999997 0.7981199999999999
- joint leg_BR_weld: origin xyz=1.9558 3.7830399999999997 0.83622 -> xyz=1.9558 3.7830399999999997 0.7981199999999999
- joint leg_FL_weld: origin xyz=-0.1524 -0.1524 0.83622 -> xyz=-0.1524 -0.1524 0.7981199999999999
- joint leg_FR_weld: origin xyz=1.9558 -0.1524 0.83622 -> xyz=1.9558 -0.1524 0.7981199999999999
- joint table_weld: origin xyz=0.9017 1.8153199999999998 -0.31933999999999996 -> xyz=0.9017 1.81532 -0.31933999999999996

File: assets/system_model/installation_capsules.urdf (robot description, URDF)
Before this commit: robot aris_system_model_capsule, 186 links, 185 joints
Links:
- link leg_BL: geometry collision box size=0.0762 0.0761999999999996 1.6509999999999998; visual box size=0.0762 0.0761999999999996 1.6509999999999998
- link leg_BR: geometry collision box size=0.07620000000000005 0.0761999999999996 1.6509999999999998; visual box size=0.07620000000000005 0.0761999999999996 1.6509999999999998
- link leg_FL: geometry collision box size=0.0762 0.0762 1.6509999999999998; visual box size=0.0762 0.0762 1.6509999999999998
- link leg_FR: geometry collision box size=0.07620000000000005 0.0762 1.6509999999999998; visual box size=0.07620000000000005 0.0762 1.6509999999999998
- link table: geometry collision box size=2.032 3.8592400000000002 0.6346799999999999; visual box size=2.032 3.8592400000000002 0.6346799999999999
Joints:
- joint leg_BL_weld: origin xyz=-0.1524 3.7830399999999997 0.83622 -> xyz=-0.1524 3.7830399999999997 0.7981199999999999
- joint leg_BR_weld: origin xyz=1.9558 3.7830399999999997 0.83622 -> xyz=1.9558 3.7830399999999997 0.7981199999999999
- joint leg_FL_weld: origin xyz=-0.1524 -0.1524 0.83622 -> xyz=-0.1524 -0.1524 0.7981199999999999
- joint leg_FR_weld: origin xyz=1.9558 -0.1524 0.83622 -> xyz=1.9558 -0.1524 0.7981199999999999
- joint table_weld: origin xyz=0.9017 1.8153199999999998 -0.31933999999999996 -> xyz=0.9017 1.81532 -0.31933999999999996

Commit message: model the seam frame: the two half-cages meet at the middle arm row, and v19 fails on it
Pete Werner, on the real hardware: "there are a few bars on the real hardware
that are not in our model.  they are supports in the middle, I think the
half-table drawing had them.  the real thing is essentially the two halves next
to each other."

THE ARITHMETIC THAT SAYS WHERE THE SEAM IS.  The drawing describes ONE
self-supporting cage, 218.44 x 208.28 cm.  Two of them butted outer face to
outer face are 4165.60 mm; this model's frame is 4011.64.  The difference,
153.96, is one doubled 3 in end frame (152.4) to within 1.56 mm — and laying
each half flush with this model's own frame ends puts its seam-side END RAIL
within 0.78 mm of the MIDDLE RUNWAY this model already builds there.

So the middle runway IS the two butted end rails.  That steel is not missing
and is not added twice; seam_bodies() builds no rail and the tests refuse one.
What WAS missing is what holds those rails up: four 3 in posts, cut 1651.0 —
the same cut as a corner leg — standing from the tabletop to the runway
underside at the frame's own x corners, straddling y = 1815.32.  Exactly the
mid-span legs OPEN_QUESTIONS['cage_legs'] said were almost certainly required.

77 static bodies -> 81.  check_system_model.py ALL PASS.

WHAT IT COSTS (scripts/seam_impact.py, h = 0.970; the certified static set is
UNCHANGED — wiring the seam in is a re-certification and it waits on a photo):

  * PARKS.  Only arms 31 and 71 ever offend — the middle row, whose J1 axes are
    ON the seam plane.  Q_PARK_PROPOSED scrapes STATIC_MARGIN by 0.9 mm and
    misses FRAME_FLOOR by 12.1.  stage_parks[2] and [6] are 35.3 mm INSIDE the
    steel.  Seven of eight stages hold a park that fails a floor.
  * CERTIFIED AREA.  16 184 -> 16 019 live cells (-165, -1.02 %), all of them
    31's and 71's, all at the canvas x extremes on the seam row.  The
    1.50 x 3.64 m hole-free block is UNCHANGED.  Lower bound: only the draw
    pose is on disk.
  * v19, whole merged timeline: frame clearance -59.4 mm, arm 31 at t = 13.94 s,
    FAIL arms [31, 71].  Everything else still passes.

The corner brace plates are carried as a question, not as geometry: as AABBs
they overlap the posts they bolt to, the model's own corner legs have never had
them, and they sit 450 mm above anything reachable.

NOT PHOTOGRAPHED.  Five assumptions ride on this — OPEN_QUESTIONS['seam_frame']
and docs/BUILD_SHEET.md section 9 list them and the two photographs that settle
them.  No gate constant, tool transform or layout grid value moved.

Co-Authored-By: Claude Opus 5 <noreply@anthropic.com>
Claude-Session: https://claude.ai/code/session_01TYL3Cueh7sskNU8Uz21h7x

File: assets/system_model/environment.urdf (robot description, URDF)
Before this commit: robot aris_system_model_env, 78 links, 77 joints
Links:
- added link seam_post_NE; collision box size=0.07620000000000005 0.07620000000000005 1.6509999999999998; visual box size=0.07620000000000005 0.07620000000000005 1.6509999999999998
- added link seam_post_NW; collision box size=0.0762 0.07620000000000005 1.6509999999999998; visual box size=0.0762 0.07620000000000005 1.6509999999999998
- added link seam_post_SE; collision box size=0.07620000000000005 0.07620000000000005 1.6509999999999998; visual box size=0.07620000000000005 0.07620000000000005 1.6509999999999998
- added link seam_post_SW; collision box size=0.0762 0.07620000000000005 1.6509999999999998; visual box size=0.0762 0.07620000000000005 1.6509999999999998
Joints:
- added joint seam_post_NE_weld: type fixed, parent world, child seam_post_NE, origin xyz=1.9558 1.85342 0.7981199999999999
- added joint seam_post_NW_weld: type fixed, parent world, child seam_post_NW, origin xyz=-0.1524 1.85342 0.7981199999999999
- added joint seam_post_SE_weld: type fixed, parent world, child seam_post_SE, origin xyz=1.9558 1.77722 0.7981199999999999
- added joint seam_post_SW_weld: type fixed, parent world, child seam_post_SW, origin xyz=-0.1524 1.77722 0.7981199999999999

File: assets/system_model/installation.urdf (robot description, URDF)
Before this commit: robot aris_system_model, 186 links, 185 joints
Links:
- added link seam_post_NE; collision box size=0.07620000000000005 0.07620000000000005 1.6509999999999998; visual box size=0.07620000000000005 0.07620000000000005 1.6509999999999998
- added link seam_post_NW; collision box size=0.0762 0.07620000000000005 1.6509999999999998; visual box size=0.0762 0.07620000000000005 1.6509999999999998
- added link seam_post_SE; collision box size=0.07620000000000005 0.07620000000000005 1.6509999999999998; visual box size=0.07620000000000005 0.07620000000000005 1.6509999999999998
- added link seam_post_SW; collision box size=0.0762 0.07620000000000005 1.6509999999999998; visual box size=0.0762 0.07620000000000005 1.6509999999999998
Joints:
- added joint seam_post_NE_weld: type fixed, parent world, child seam_post_NE, origin xyz=1.9558 1.85342 0.7981199999999999
- added joint seam_post_NW_weld: type fixed, parent world, child seam_post_NW, origin xyz=-0.1524 1.85342 0.7981199999999999
- added joint seam_post_SE_weld: type fixed, parent world, child seam_post_SE, origin xyz=1.9558 1.77722 0.7981199999999999
- added joint seam_post_SW_weld: type fixed, parent world, child seam_post_SW, origin xyz=-0.1524 1.77722 0.7981199999999999

File: assets/system_model/installation_capsules.urdf (robot description, URDF)
Before this commit: robot aris_system_model_capsule, 186 links, 185 joints
Links:
- added link seam_post_NE; collision box size=0.07620000000000005 0.07620000000000005 1.6509999999999998; visual box size=0.07620000000000005 0.07620000000000005 1.6509999999999998
- added link seam_post_NW; collision box size=0.0762 0.07620000000000005 1.6509999999999998; visual box size=0.0762 0.07620000000000005 1.6509999999999998
- added link seam_post_SE; collision box size=0.07620000000000005 0.07620000000000005 1.6509999999999998; visual box size=0.07620000000000005 0.07620000000000005 1.6509999999999998
- added link seam_post_SW; collision box size=0.0762 0.07620000000000005 1.6509999999999998; visual box size=0.0762 0.07620000000000005 1.6509999999999998
Joints:
- added joint seam_post_NE_weld: type fixed, parent world, child seam_post_NE, origin xyz=1.9558 1.85342 0.7981199999999999
- added joint seam_post_NW_weld: type fixed, parent world, child seam_post_NW, origin xyz=-0.1524 1.85342 0.7981199999999999
- added joint seam_post_SE_weld: type fixed, parent world, child seam_post_SE, origin xyz=1.9558 1.77722 0.7981199999999999
- added joint seam_post_SW_weld: type fixed, parent world, child seam_post_SW, origin xyz=-0.1524 1.77722 0.7981199999999999

File: assets/system_model/installation_fatfingers.urdf (robot description, URDF)
Before this commit: robot aris_system_model_fatfingers, 186 links, 185 joints
Links:
- added link seam_post_NE; collision box size=0.07620000000000005 0.07620000000000005 1.6509999999999998; visual box size=0.07620000000000005 0.07620000000000005 1.6509999999999998
- added link seam_post_NW; collision box size=0.0762 0.07620000000000005 1.6509999999999998; visual box size=0.0762 0.07620000000000005 1.6509999999999998
- added link seam_post_SE; collision box size=0.07620000000000005 0.07620000000000005 1.6509999999999998; visual box size=0.07620000000000005 0.07620000000000005 1.6509999999999998
- added link seam_post_SW; collision box size=0.0762 0.07620000000000005 1.6509999999999998; visual box size=0.0762 0.07620000000000005 1.6509999999999998
Joints:
- added joint seam_post_NE_weld: type fixed, parent world, child seam_post_NE, origin xyz=1.9558 1.85342 0.7981199999999999
- added joint seam_post_NW_weld: type fixed, parent world, child seam_post_NW, origin xyz=-0.1524 1.85342 0.7981199999999999
- added joint seam_post_SE_weld: type fixed, parent world, child seam_post_SE, origin xyz=1.9558 1.77722 0.7981199999999999
- added joint seam_post_SW_weld: type fixed, parent world, child seam_post_SW, origin xyz=-0.1524 1.77722 0.7981199999999999

Commit message: diag: why stage A's follower keeps nothing, measured on arm 31
Rebuilds stage A of the leader/follower pattern at split +0.15 -- the same
DP, the same role order, the same trajectory rooms -- and stops at the
follower with the most offered ink (arm 31, 2.144 m, the only stage-A
follower the DP gives ink to at this split).  Measures, per leader room
separately: the follower's INK pose by pose, every pen-up LEG the timeline
would need, the five hypotheses, and what the follower would keep if the
same-row leader's bag were capped by reach.  Read-only on the planner;
scene on meshcat 7007 and out/lf_follower_diag.html.

Co-Authored-By: Claude Opus 5 <noreply@anthropic.com>
Claude-Session: https://claude.ai/code/session_01TYL3Cueh7sskNU8Uz21h7x

File: assets/system_model/environment.urdf (robot description, URDF)
Before this commit: robot aris_system_model_env, 82 links, 81 joints
Links:
- removed link seam_post_NE
- removed link seam_post_NW
- removed link seam_post_SE
- removed link seam_post_SW
- added link seam_bar_E; collision box size=0.07620000000000005 0.1524000000000001 1.6509999999999998; visual box size=0.07620000000000005 0.1524000000000001 1.6509999999999998
- added link seam_bar_W; collision box size=0.0762 0.1524000000000001 1.6509999999999998; visual box size=0.0762 0.1524000000000001 1.6509999999999998
Joints:
- removed joint seam_post_NE_weld
- removed joint seam_post_NW_weld
- removed joint seam_post_SE_weld
- removed joint seam_post_SW_weld
- added joint seam_bar_E_weld: type fixed, parent world, child seam_bar_E, origin xyz=1.9558 1.81532 0.7981199999999999
- added joint seam_bar_W_weld: type fixed, parent world, child seam_bar_W, origin xyz=-0.1524 1.81532 0.7981199999999999

File: assets/system_model/installation.urdf (robot description, URDF)
Before this commit: robot aris_system_model, 190 links, 189 joints
Links:
- removed link seam_post_NE
- removed link seam_post_NW
- removed link seam_post_SE
- removed link seam_post_SW
- added link seam_bar_E; collision box size=0.07620000000000005 0.1524000000000001 1.6509999999999998; visual box size=0.07620000000000005 0.1524000000000001 1.6509999999999998
- added link seam_bar_W; collision box size=0.0762 0.1524000000000001 1.6509999999999998; visual box size=0.0762 0.1524000000000001 1.6509999999999998
Joints:
- removed joint seam_post_NE_weld
- removed joint seam_post_NW_weld
- removed joint seam_post_SE_weld
- removed joint seam_post_SW_weld
- added joint seam_bar_E_weld: type fixed, parent world, child seam_bar_E, origin xyz=1.9558 1.81532 0.7981199999999999
- added joint seam_bar_W_weld: type fixed, parent world, child seam_bar_W, origin xyz=-0.1524 1.81532 0.7981199999999999

File: assets/system_model/installation_capsules.urdf (robot description, URDF)
Before this commit: robot aris_system_model_capsule, 190 links, 189 joints
Links:
- removed link seam_post_NE
- removed link seam_post_NW
- removed link seam_post_SE
- removed link seam_post_SW
- added link seam_bar_E; collision box size=0.07620000000000005 0.1524000000000001 1.6509999999999998; visual box size=0.07620000000000005 0.1524000000000001 1.6509999999999998
- added link seam_bar_W; collision box size=0.0762 0.1524000000000001 1.6509999999999998; visual box size=0.0762 0.1524000000000001 1.6509999999999998
Joints:
- removed joint seam_post_NE_weld
- removed joint seam_post_NW_weld
- removed joint seam_post_SE_weld
- removed joint seam_post_SW_weld
- added joint seam_bar_E_weld: type fixed, parent world, child seam_bar_E, origin xyz=1.9558 1.81532 0.7981199999999999
- added joint seam_bar_W_weld: type fixed, parent world, child seam_bar_W, origin xyz=-0.1524 1.81532 0.7981199999999999

File: assets/system_model/installation_fatfingers.urdf (robot description, URDF)
Before this commit: robot aris_system_model_fatfingers, 190 links, 189 joints
Links:
- removed link seam_post_NE
- removed link seam_post_NW
- removed link seam_post_SE
- removed link seam_post_SW
- added link seam_bar_E; collision box size=0.07620000000000005 0.1524000000000001 1.6509999999999998; visual box size=0.07620000000000005 0.1524000000000001 1.6509999999999998
- added link seam_bar_W; collision box size=0.0762 0.1524000000000001 1.6509999999999998; visual box size=0.0762 0.1524000000000001 1.6509999999999998
Joints:
- removed joint seam_post_NE_weld
- removed joint seam_post_NW_weld
- removed joint seam_post_SE_weld
- removed joint seam_post_SW_weld
- added joint seam_bar_E_weld: type fixed, parent world, child seam_bar_E, origin xyz=1.9558 1.81532 0.7981199999999999
- added joint seam_bar_W_weld: type fixed, parent world, child seam_bar_W, origin xyz=-0.1524 1.81532 0.7981199999999999
